Commit message: adding tool, not functionnel in moveit

File: denso_ros2_ws/src/denso_robot_drivers_ros2/denso_robot_descriptions/urdf/denso_robot.urdf.xacro (robot description, xacro)
@@ -24,3 +24,28 @@
      send_format="$(arg send_format)"
      recv_format="$(arg recv_format)" />
+   <link name="$(arg namespace)tool_link">
+    <visual>
+      <origin xyz="0 0 0" rpy="0 0 0" />
+      <geometry>
+        <mesh filename="file://$(find denso_robot_descriptions)/robots/$(arg model)/meshes/EffecteurV1.STL" scale="0.001 0.001 0.001"/>
+      </geometry>
+      <material name="grey">
+        <color rgba="0.5 0.5 0.5 1.0"/>
+      </material>
+    </visual>
+    <collision>
+      <origin xyz="0 0 0" rpy="0 0 0" />
+      <geometry>
+        <mesh filename="file://$(find denso_robot_descriptions)/robots/$(arg model)/meshes/EffecteurV1.STL" scale="0.001 0.001 0.001"/>
+      </geometry>
+    </collision>
+    <inertial>
+       <mass value="0.5" /> <origin xyz="0 0 0.05" rpy="0 0 0" /> <inertia ixx="0.001" ixy="0.0" ixz="0.0" iyy="0.001" iyz="0.0" izz="0.001" />
+    </inertial>
+  </link>
+  <joint name="$(arg namespace)tool_joint" type="fixed">
+    <parent link="$(arg namespace)J6" />
+    <child link="$(arg namespace)tool_link" />
+    <origin xyz="0 0 0" rpy="0 0 0" />
+  </joint>
 </robot>

File: denso_ros2_ws/src/denso_robot_drivers_ros2/denso_robot_moveit_config/robots/vs060/srdf/denso_robot_macro.srdf.xacro (robot description, xacro)
@@ -32,4 +32,5 @@
 	<disable_collisions link1="$(arg namespace)J3" link2="$(arg namespace)J5" reason="Never"/>
 	<disable_collisions link1="$(arg namespace)J4" link2="$(arg namespace)J5" reason="Adjacent"/>
+  <disable_collisions link1="$(arg namespace)J6" link2="$(arg namespace)tool_link" reason="Attached by fixed joint" />
   </xacro:macro>
 </robot>

Commit message: tool position used in moveit

File: denso_ros2_ws/src/denso_robot_drivers_ros2/denso_robot_descriptions/urdf/denso_robot.urdf.xacro (robot description, xacro)
@@ -26,5 +26,5 @@
    <link name="$(arg namespace)tool_link">
     <visual>
-      <origin xyz="0 0 0" rpy="0 0 0" />
+      <origin xyz="0 0 -0.207" rpy="0 0 0" />
       <geometry>
         <mesh filename="file://$(find denso_robot_descriptions)/robots/$(arg model)/meshes/EffecteurV1.STL" scale="0.001 0.001 0.001"/>
@@ -35,5 +35,5 @@
     </visual>
     <collision>
-      <origin xyz="0 0 0" rpy="0 0 0" />
+      <origin xyz="0 0 -0.207" rpy="0 0 0" />
       <geometry>
         <mesh filename="file://$(find denso_robot_descriptions)/robots/$(arg model)/meshes/EffecteurV1.STL" scale="0.001 0.001 0.001"/>
@@ -41,5 +41,5 @@
     </collision>
     <inertial>
-       <mass value="0.5" /> <origin xyz="0 0 0.05" rpy="0 0 0" /> <inertia ixx="0.001" ixy="0.0" ixz="0.0" iyy="0.001" iyz="0.0" izz="0.001" />
+       <mass value="0.5" /> <origin xyz="0 0 0.1" rpy="0 0 0" /> <inertia ixx="0.001" ixy="0.0" ixz="0.0" iyy="0.001" iyz="0.0" izz="0.001" />
     </inertial>
   </link>
@@ -47,5 +47,5 @@
     <parent link="$(arg namespace)J6" />
     <child link="$(arg namespace)tool_link" />
-    <origin xyz="0 0 0" rpy="0 0 0" />
+    <origin xyz="0 0 0.207" rpy="0 0 0" />
   </joint>
 </robot>

File: denso_ros2_ws/src/denso_robot_drivers_ros2/denso_robot_moveit_config/robots/vs060/srdf/denso_robot_macro.srdf.xacro (robot description, xacro)
@@ -11,12 +11,15 @@
     <!--CHAINS - When a chain is specified, all the links along the chain (including endpoints) are included in the group. Additionally, all the joints that are parents to included links are also included. This means that joints along the chain and the parent joint of the base link are included in the group-->
     <!--SUBGROUPS - Groups can also be formed by referencing to already defined group names-->
-    <group name="${namespace}arm">
-		<joint name="$(arg namespace)joint_1"/>
-		<joint name="$(arg namespace)joint_2"/>
-		<joint name="$(arg namespace)joint_3"/>
-		<joint name="$(arg namespace)joint_4"/>
-		<joint name="$(arg namespace)joint_5"/>
-		<joint name="$(arg namespace)joint_6"/>
-	</group>
+    <!-- <group name="${namespace}arm">
+      <joint name="$(arg namespace)joint_1"/>
+      <joint name="$(arg namespace)joint_2"/>
+      <joint name="$(arg namespace)joint_3"/>
+      <joint name="$(arg namespace)joint_4"/>
+      <joint name="$(arg namespace)joint_5"/>
+      <joint name="$(arg namespace)joint_6"/>
+    </group> -->
+    <group name="arm">
+      <chain base_link="$(arg namespace)base_link" tip_link="$(arg namespace)tool_link"/>
+    </group>
     <!--GROUP STATES - Purpose - Define a named state for a particular group, in terms of joint values. This is useful to define states like 'folded arms'-->
     <!--END EFFECTOR - Purpose - Represent information about an end effector.-->

Commit message: select tool on start

File: denso_ros2_ws/src/denso_robot_drivers_ros2/denso_robot_descriptions/urdf/denso_robot.urdf.xacro (robot description, xacro)
@@ -1,12 +1,9 @@
 <?xml version="1.0"?>
 <robot xmlns:xacro="http://wiki.ros.org/xacro" name="$(arg model)">
-   <!-- robot name parameter -->
+   <xacro:arg name="tool" default="none"/>
    <xacro:arg name="model" default="denso_robot"/>
-   <!-- import main macro -->
    <xacro:include filename="$(find denso_robot_descriptions)/robots/$(arg model)/urdf/denso_robot_macro.xacro"/>
-   <!-- parameters -->
    <xacro:arg name="namespace" default="" />
    <xacro:arg name="transmission_hw_interface" default=""/>
-   <!-- ros2_control related parameters -->
    <xacro:arg name="verbose" default="false" />
    <xacro:arg name="sim" default="false" />
@@ -14,5 +11,4 @@
    <xacro:arg name="send_format" default="288" />
    <xacro:arg name="recv_format" default="292" />
-   <!-- arm -->
    <xacro:denso_robot
      model="$(arg model)"
@@ -24,28 +20,55 @@
      send_format="$(arg send_format)"
      recv_format="$(arg recv_format)" />
-   <link name="$(arg namespace)tool_link">
-    <visual>
-      <origin xyz="0 0 -0.207" rpy="0 0 0" />
-      <geometry>
-        <mesh filename="file://$(find denso_robot_descriptions)/robots/$(arg model)/meshes/EffecteurV1.STL" scale="0.001 0.001 0.001"/>
-      </geometry>
-      <material name="grey">
-        <color rgba="0.5 0.5 0.5 1.0"/>
-      </material>
-    </visual>
-    <collision>
-      <origin xyz="0 0 -0.207" rpy="0 0 0" />
-      <geometry>
-        <mesh filename="file://$(find denso_robot_descriptions)/robots/$(arg model)/meshes/EffecteurV1.STL" scale="0.001 0.001 0.001"/>
-      </geometry>
-    </collision>
-    <inertial>
-       <mass value="0.5" /> <origin xyz="0 0 0.1" rpy="0 0 0" /> <inertia ixx="0.001" ixy="0.0" ixz="0.0" iyy="0.001" iyz="0.0" izz="0.001" />
-    </inertial>
-  </link>
-  <joint name="$(arg namespace)tool_joint" type="fixed">
-    <parent link="$(arg namespace)J6" />
-    <child link="$(arg namespace)tool_link" />
-    <origin xyz="0 0 0.207" rpy="0 0 0" />
-  </joint>
+   <xacro:if value="${'$(arg tool)' == 'effecteur_v1'}">
+     <link name="$(arg namespace)tool_link">
+      <visual>
+        <origin xyz="0 0 -0.207" rpy="0 0 0" />
+        <geometry>
+          <mesh filename="file://$(find denso_robot_descriptions)/robots/$(arg model)/meshes/EffecteurV1.STL" scale="0.001 0.001 0.001"/>
+        </geometry>
+        <material name="grey">
+          <color rgba="0.5 0.5 0.5 1.0"/>
+        </material>
+      </visual>
+      <collision>
+        <origin xyz="0 0 -0.207" rpy="0 0 0" />
+        <geometry>
+          <mesh filename="file://$(find denso_robot_descriptions)/robots/$(arg model)/meshes/EffecteurV1.STL" scale="0.001 0.001 0.001"/>
+        </geometry>
+      </collision>
+      <inertial>
+         <mass value="0.5" /> <origin xyz="0 0 0.1" rpy="0 0 0" /> <inertia ixx="0.001" ixy="0.0" ixz="0.0" iyy="0.001" iyz="0.0" izz="0.001" />
+      </inertial>
+     </link>
+     <joint name="$(arg namespace)tool_joint" type="fixed">
+      <parent link="$(arg namespace)J6" />
+      <child link="$(arg namespace)tool_link" />
+      <origin xyz="0 0 0.207" rpy="0 0 0" />
+     </joint>
+   </xacro:if>
+   <xacro:if value="${'$(arg tool)' == 'effecteur_test'}">
+     <link name="$(arg namespace)tool_link">
+      <visual>
+        <origin xyz="0 0 0" rpy="0 0 0" /> <geometry>
+          <mesh filename="file://$(find denso_robot_descriptions)/robots/$(arg model)/meshes/EffecteurTest.STL" scale="0.001 0.001 0.001"/>
+        </geometry>
+        <material name="blue">
+          <color rgba="0.0 0.0 0.8 1.0"/> </material>
+      </visual>
+      <collision>
+        <origin xyz="0 0 0.0" rpy="0 0 0" /> <geometry>
+          <mesh filename="file://$(find denso_robot_descriptions)/robots/$(arg model)/meshes/EffecteurTest.STL" scale="0.001 0.001 0.001"/>
+        </geometry>
+      </collision>
+      <inertial>
+         <mass value="0.8" />
+         <origin xyz="0 0 0.05" rpy="0 0 0" />
+         <inertia ixx="0.002" ixy="0.0" ixz="0.0" iyy="0.002" iyz="0.0" izz="0.002" />
+      </inertial>
+     </link>
+     <joint name="$(arg namespace)tool_joint" type="fixed">
+      <parent link="$(arg namespace)J6" />
+      <child link="$(arg namespace)tool_link" />
+      <origin xyz="0 0 0.0" rpy="0 0 0" /> </joint>
+   </xacro:if>
 </robot>

File: denso_ros2_ws/src/denso_robot_drivers_ros2/denso_robot_moveit_config/robots/vs060/srdf/denso_robot_macro.srdf.xacro (robot description, xacro)
@@ -1,39 +1,24 @@
 <?xml version="1.0" encoding="UTF-8"?>
 <robot xmlns:xacro="http://wiki.ros.org/xacro">
-<!--This does not replace URDF, and is not an extension of URDF.
-    This is a format for representing semantic information about the robot structure.
-    A URDF file must exist for this robot as well, where the joints and the links that are referenced are defined
--->
-  <xacro:macro name="denso_robot_srdf" params="name namespace">
-    <!--GROUPS - Representation of a set of joints and links. This can be useful for specifying DOF to plan for, defining arms, end effectors, etc-->
-    <!--LINKS - When a link is specified, the parent joint of that link (if it exists) is automatically included-->
-    <!--JOINTS - When a joint is specified, the child link of that joint (which will always exist) is automatically included-->
-    <!--CHAINS - When a chain is specified, all the links along the chain (including endpoints) are included in the group. Additionally, all the joints that are parents to included links are also included. This means that joints along the chain and the parent joint of the base link are included in the group-->
-    <!--SUBGROUPS - Groups can also be formed by referencing to already defined group names-->
-    <!-- <group name="${namespace}arm">
-      <joint name="$(arg namespace)joint_1"/>
-      <joint name="$(arg namespace)joint_2"/>
-      <joint name="$(arg namespace)joint_3"/>
-      <joint name="$(arg namespace)joint_4"/>
-      <joint name="$(arg namespace)joint_5"/>
-      <joint name="$(arg namespace)joint_6"/>
-    </group> -->
+  <xacro:macro name="denso_robot_srdf" params="name namespace tool">
     <group name="arm">
-      <chain base_link="$(arg namespace)base_link" tip_link="$(arg namespace)tool_link"/>
+      <xacro:if value="${tool == 'none'}">
+        <chain base_link="$(arg namespace)base_link" tip_link="$(arg namespace)J6"/>
+      </xacro:if>
+      <xacro:if value="${tool != 'none'}">
+        <chain base_link="$(arg namespace)base_link" tip_link="$(arg namespace)tool_link"/>
+      </xacro:if>
     </group>
-    <!--GROUP STATES - Purpose - Define a named state for a particular group, in terms of joint values. This is useful to define states like 'folded arms'-->
-    <!--END EFFECTOR - Purpose - Represent information about an end effector.-->
-    <!--VIRTUAL JOINT - Purpose - this element defines a virtual joint between a robot link and an external frame of reference (considered fixed with respect to the robot)-->
     <virtual_joint name="${namespace}fixed_base" type="fixed" parent_frame="world" child_link="${namespace}base_link" />
-    <!--DISABLE COLLISIONS - By default it is assumed that any link of the robot could potentially come into collision with any other link in the robot. This tag disables collision checking between a specified pair of links. -->
-	<disable_collisions link1="$(arg namespace)J6" link2="$(arg namespace)J3" reason="Never"/>
-	<disable_collisions link1="$(arg namespace)J6" link2="$(arg namespace)J5" reason="Adjacent"/>
-	<disable_collisions link1="$(arg namespace)J1" link2="$(arg namespace)J2" reason="Adjacent"/>
-	<disable_collisions link1="$(arg namespace)J1" link2="$(arg namespace)base_link" reason="Adjacent"/>
-	<disable_collisions link1="$(arg namespace)J2" link2="$(arg namespace)J3" reason="Adjacent"/>
-	<disable_collisions link1="$(arg namespace)J3" link2="$(arg namespace)J4" reason="Adjacent"/>
-	<disable_collisions link1="$(arg namespace)J3" link2="$(arg namespace)J5" reason="Never"/>
-	<disable_collisions link1="$(arg namespace)J4" link2="$(arg namespace)J5" reason="Adjacent"/>
-  <disable_collisions link1="$(arg namespace)J6" link2="$(arg namespace)tool_link" reason="Attached by fixed joint" />
+    <disable_collisions link1="$(arg namespace)J6" link2="$(arg namespace)J3" reason="Never"/>
+    <disable_collisions link1="$(arg namespace)J6" link2="$(arg namespace)J5" reason="Adjacent"/>
+    <disable_collisions link1="$(arg namespace)J1" link2="$(arg namespace)J2" reason="Adjacent"/>
+    <disable_collisions link1="$(arg namespace)J1" link2="$(arg namespace)base_link" reason="Adjacent"/>
+    <disable_collisions link1="$(arg namespace)J2" link2="$(arg namespace)J3" reason="Adjacent"/>
+    <disable_collisions link1="$(arg namespace)J3" link2="$(arg namespace)J4" reason="Adjacent"/> <disable_collisions link1="$(arg namespace)J3" link2="$(arg namespace)J5" reason="Never"/>
+    <disable_collisions link1="$(arg namespace)J4" link2="$(arg namespace)J5" reason="Adjacent"/>
+    <xacro:if value="${tool != 'none'}">
+      <disable_collisions link1="$(arg namespace)J6" link2="$(arg namespace)tool_link" reason="Attached by fixed joint" />
+    </xacro:if>
   </xacro:macro>
 </robot>

File: denso_ros2_ws/src/denso_robot_drivers_ros2/denso_robot_moveit_config/srdf/denso_robot.srdf.xacro (robot description, xacro)
@@ -1,9 +1,8 @@
 <?xml version="1.0" encoding="UTF-8"?>
 <robot xmlns:xacro="http://wiki.ros.org/xacro" name="$(arg model)">
-  <!-- robot name parameter -->
   <xacro:arg name="model" default="denso_robot"/>
-  <!-- parameters -->
   <xacro:arg name="namespace" default="" />
+  <xacro:arg name="tool" default="none" />
   <xacro:include filename="$(find denso_robot_moveit_config)/robots/$(arg model)/srdf/denso_robot_macro.srdf.xacro"/>
-  <xacro:denso_robot_srdf name="$(arg namespace)$(arg model)" namespace="$(arg namespace)"/>
+  <xacro:denso_robot_srdf name="$(arg namespace)$(arg model)" namespace="$(arg namespace)" tool="$(arg tool)"/>
 </robot>

Commit message: adding tool on existing denso robot

File: denso_ros2_ws/src/denso_robot_drivers_ros2/denso_robot_descriptions/urdf/denso_robot.urdf.xacro (robot description, xacro)
@@ -20,55 +20,19 @@
      send_format="$(arg send_format)"
      recv_format="$(arg recv_format)" />
-   <xacro:if value="${'$(arg tool)' == 'effecteur_v1'}">
-     <link name="$(arg namespace)tool_link">
-      <visual>
-        <origin xyz="0 0 -0.207" rpy="0 0 0" />
-        <geometry>
-          <mesh filename="file://$(find denso_robot_descriptions)/robots/$(arg model)/meshes/EffecteurV1.STL" scale="0.001 0.001 0.001"/>
-        </geometry>
-        <material name="grey">
-          <color rgba="0.5 0.5 0.5 1.0"/>
-        </material>
-      </visual>
-      <collision>
-        <origin xyz="0 0 -0.207" rpy="0 0 0" />
-        <geometry>
-          <mesh filename="file://$(find denso_robot_descriptions)/robots/$(arg model)/meshes/EffecteurV1.STL" scale="0.001 0.001 0.001"/>
-        </geometry>
-      </collision>
-      <inertial>
-         <mass value="0.5" /> <origin xyz="0 0 0.1" rpy="0 0 0" /> <inertia ixx="0.001" ixy="0.0" ixz="0.0" iyy="0.001" iyz="0.0" izz="0.001" />
-      </inertial>
-     </link>
-     <joint name="$(arg namespace)tool_joint" type="fixed">
-      <parent link="$(arg namespace)J6" />
-      <child link="$(arg namespace)tool_link" />
-      <origin xyz="0 0 0.207" rpy="0 0 0" />
-     </joint>
+   <!-- <xacro:unless value="${'$(arg tool)' == 'none'}">
+     <xacro:include filename="$(find denso_robot_descriptions)/tools/$(arg tool)/$(arg tool).xacro"/>
+     <xacro:call macro="$(arg tool)" namespace="$(arg namespace)" parent_link="$(arg namespace)J6" />
+   </xacro:unless>
+    -->
+   <xacro:property name="tool_parent_link" value="$(arg namespace)J6" />
+   <xacro:if value="${'$(arg model)' == 'hsr065a1_n32'}">
+     <xacro:property name="tool_parent_link" value="$(arg namespace)J4" />
    </xacro:if>
-   <xacro:if value="${'$(arg tool)' == 'effecteur_test'}">
-     <link name="$(arg namespace)tool_link">
-      <visual>
-        <origin xyz="0 0 0" rpy="0 0 0" /> <geometry>
-          <mesh filename="file://$(find denso_robot_descriptions)/robots/$(arg model)/meshes/EffecteurTest.STL" scale="0.001 0.001 0.001"/>
-        </geometry>
-        <material name="blue">
-          <color rgba="0.0 0.0 0.8 1.0"/> </material>
-      </visual>
-      <collision>
-        <origin xyz="0 0 0.0" rpy="0 0 0" /> <geometry>
-          <mesh filename="file://$(find denso_robot_descriptions)/robots/$(arg model)/meshes/EffecteurTest.STL" scale="0.001 0.001 0.001"/>
-        </geometry>
-      </collision>
-      <inertial>
-         <mass value="0.8" />
-         <origin xyz="0 0 0.05" rpy="0 0 0" />
-         <inertia ixx="0.002" ixy="0.0" ixz="0.0" iyy="0.002" iyz="0.0" izz="0.002" />
-      </inertial>
-     </link>
-     <joint name="$(arg namespace)tool_joint" type="fixed">
-      <parent link="$(arg namespace)J6" />
-      <child link="$(arg namespace)tool_link" />
-      <origin xyz="0 0 0.0" rpy="0 0 0" /> </joint>
-   </xacro:if>
+   <!-- <xacro:if value="${'$(arg model)' == 'nom_de_votre_robot_5_axes'}">
+     <xacro:property name="tool_parent_link" value="$(arg namespace)J5" />
+   </xacro:if> -->
+   <xacro:unless value="${'$(arg tool)' == 'none'}">
+     <xacro:include filename="$(find denso_robot_descriptions)/tools/$(arg tool)/$(arg tool).xacro"/>
+     <xacro:call macro="$(arg tool)" namespace="$(arg namespace)" parent_link="${tool_parent_link}" />
+   </xacro:unless>
 </robot>

File: denso_ros2_ws/src/denso_robot_drivers_ros2/denso_robot_moveit_config/robots/cobotta/srdf/denso_robot_macro.srdf.xacro (robot description, xacro)
@@ -5,5 +5,5 @@
     A URDF file must exist for this robot as well, where the joints and the links that are referenced are defined
 -->
-  <xacro:macro name="denso_robot_srdf" params="name namespace">
+  <xacro:macro name="denso_robot_srdf" params="name namespace tool">
     <!--GROUPS - Representation of a set of joints and links. This can be useful for specifying DOF to plan for, defining arms, end effectors, etc-->
     <!--LINKS - When a link is specified, the parent joint of that link (if it exists) is automatically included-->
@@ -18,4 +18,10 @@
 		<joint name="$(arg namespace)joint_5"/>
 		<joint name="$(arg namespace)joint_6"/>
+    <xacro:if value="${tool == 'none'}">
+      <chain base_link="$(arg namespace)base_link" tip_link="$(arg namespace)J6"/>
+    </xacro:if>
+    <xacro:if value="${tool != 'none'}">
+      <chain base_link="$(arg namespace)base_link" tip_link="$(arg namespace)tool_link"/>
+    </xacro:if>
 	</group>
     <!--GROUP STATES - Purpose - Define a named state for a particular group, in terms of joint values. This is useful to define states like 'folded arms'-->
@@ -32,4 +38,7 @@
 	<disable_collisions link1="$(arg namespace)J3" link2="$(arg namespace)J5" reason="Never"/>
 	<disable_collisions link1="$(arg namespace)J4" link2="$(arg namespace)J5" reason="Adjacent"/>
+  <xacro:if value="${tool != 'none'}">
+    <disable_collisions link1="$(arg namespace)J6" link2="$(arg namespace)tool_link" reason="Attached by fixed joint" />
+  </xacro:if>
   </xacro:macro>
 </robot>

File: denso_ros2_ws/src/denso_robot_drivers_ros2/denso_robot_moveit_config/robots/hsr065a1_n32/srdf/denso_robot_macro.srdf.xacro (robot description, xacro)
@@ -5,5 +5,5 @@
     A URDF file must exist for this robot as well, where the joints and the links that are referenced are defined
 -->
-  <xacro:macro name="denso_robot_srdf" params="name namespace">
+  <xacro:macro name="denso_robot_srdf" params="name namespace tool">
     <!--GROUPS - Representation of a set of joints and links. This can be useful for specifying DOF to plan for, defining arms, end effectors, etc-->
     <!--LINKS - When a link is specified, the parent joint of that link (if it exists) is automatically included-->
@@ -16,4 +16,10 @@
 		<joint name="$(arg namespace)joint_3"/>
 		<joint name="$(arg namespace)joint_4"/>
+    <xacro:if value="${tool == 'none'}">
+      <chain base_link="$(arg namespace)base_link" tip_link="$(arg namespace)J6"/>
+    </xacro:if>
+    <xacro:if value="${tool != 'none'}">
+      <chain base_link="$(arg namespace)base_link" tip_link="$(arg namespace)tool_link"/>
+    </xacro:if>
 	</group>
     <!--GROUP STATES - Purpose - Define a named state for a particular group, in terms of joint values. This is useful to define states like 'folded arms'-->
@@ -31,4 +37,7 @@
 	<disable_collisions link1="$(arg namespace)J3" link2="$(arg namespace)J4" reason="Adjacent"/>
 	<disable_collisions link1="$(arg namespace)J4" link2="$(arg namespace)base_link" reason="Never"/>
+  <xacro:if value="${tool != 'none'}">
+      <disable_collisions link1="$(arg namespace)J6" link2="$(arg namespace)tool_link" reason="Attached by fixed joint" />
+  </xacro:if>
   </xacro:macro>
 </robot>
