Commit message: vp5243 working and not too heavy for moveit

File: denso_ros2_ws/src/denso_robot_drivers_ros2/denso_robot_descriptions/robots/vp5243/urdf/denso_robot_kinematics.xacro (robot description, xacro)
@@ -11,5 +11,5 @@
 				<origin rpy="0 0 0" xyz="0 0 0"/>
 				<geometry>
-					<mesh filename="file:///$(find denso_robot_descriptions)/robots/$(arg model)/meshes/base_link.dae" scale="1 1 1"/>
+					<mesh filename="file:///$(find denso_robot_descriptions)/robots/$(arg model)/meshes/visual/base_link.dae" scale="1 1 1"/>
 				</geometry>
 			</visual>
@@ -17,5 +17,5 @@
 				<origin rpy="0 0 0" xyz="0 0 0"/>
 				<geometry>
-					<mesh filename="file:///$(find denso_robot_descriptions)/robots/$(arg model)/meshes/base_link.dae" scale="1 1 1"/>
+					<mesh filename="file:///$(find denso_robot_descriptions)/robots/$(arg model)/meshes/collision/base_link.dae" scale="1 1 1"/>
 				</geometry>
 			</collision>
@@ -30,5 +30,5 @@
 				<origin rpy="0 0 0" xyz="0 0 0"/>
 				<geometry>
-					<mesh filename="file:///$(find denso_robot_descriptions)/robots/$(arg model)/meshes/J1.dae" scale="1 1 1"/>
+					<mesh filename="file:///$(find denso_robot_descriptions)/robots/$(arg model)/meshes/visual/J1.dae" scale="1 1 1"/>
 				</geometry>
 			</visual>
@@ -36,5 +36,5 @@
 				<origin rpy="0 0 0" xyz="0 0 0"/>
 				<geometry>
-					<mesh filename="file:///$(find denso_robot_descriptions)/robots/$(arg model)/meshes/J1.dae" scale="1 1 1"/>
+					<mesh filename="file:///$(find denso_robot_descriptions)/robots/$(arg model)/meshes/collision/J1.dae" scale="1 1 1"/>
 				</geometry>
 			</collision>
@@ -57,5 +57,5 @@
 				<origin rpy="0 0 0" xyz="0 0 0"/>
 				<geometry>
-					<mesh filename="file:///$(find denso_robot_descriptions)/robots/$(arg model)/meshes/J2.dae" scale="1 1 1"/>
+					<mesh filename="file:///$(find denso_robot_descriptions)/robots/$(arg model)/meshes/visual/J2.dae" scale="1 1 1"/>
 				</geometry>
 			</visual>
@@ -63,5 +63,5 @@
 				<origin rpy="0 0 0" xyz="0 0 0"/>
 				<geometry>
-					<mesh filename="file:///$(find denso_robot_descriptions)/robots/$(arg model)/meshes/J2.dae" scale="1 1 1"/>
+					<mesh filename="file:///$(find denso_robot_descriptions)/robots/$(arg model)/meshes/collision/J2.dae" scale="1 1 1"/>
 				</geometry>
 			</collision>
@@ -84,5 +84,5 @@
 				<origin rpy="0 0 0" xyz="0 0 0"/>
 				<geometry>
-					<mesh filename="file:///$(find denso_robot_descriptions)/robots/$(arg model)/meshes/J3.dae" scale="1 1 1"/>
+					<mesh filename="file:///$(find denso_robot_descriptions)/robots/$(arg model)/meshes/visual/J3.dae" scale="1 1 1"/>
 				</geometry>
 			</visual>
@@ -90,5 +90,5 @@
 				<origin rpy="0 0 0" xyz="0 0 0"/>
 				<geometry>
-					<mesh filename="file:///$(find denso_robot_descriptions)/robots/$(arg model)/meshes/J3.dae" scale="1 1 1"/>
+					<mesh filename="file:///$(find denso_robot_descriptions)/robots/$(arg model)/meshes/collision/J3.dae" scale="1 1 1"/>
 				</geometry>
 			</collision>
@@ -111,5 +111,5 @@
 				<origin rpy="0 0 0" xyz="0 0 0"/>
 				<geometry>
-					<mesh filename="file:///$(find denso_robot_descriptions)/robots/$(arg model)/meshes/J4.dae" scale="1 1 1"/>
+					<mesh filename="file:///$(find denso_robot_descriptions)/robots/$(arg model)/meshes/visual/J4.dae" scale="1 1 1"/>
 				</geometry>
 			</visual>
@@ -117,5 +117,5 @@
 				<origin rpy="0 0 0" xyz="0 0 0"/>
 				<geometry>
-					<mesh filename="file:///$(find denso_robot_descriptions)/robots/$(arg model)/meshes/J4.dae" scale="1 1 1"/>
+					<mesh filename="file:///$(find denso_robot_descriptions)/robots/$(arg model)/meshes/collision/J4.dae" scale="1 1 1"/>
 				</geometry>
 			</collision>
@@ -138,5 +138,5 @@
 				<origin rpy="0 0 0" xyz="0 0 0"/>
 				<geometry>
-					<mesh filename="file:///$(find denso_robot_descriptions)/robots/$(arg model)/meshes/J5.dae" scale="1 1 1"/>
+					<mesh filename="file:///$(find denso_robot_descriptions)/robots/$(arg model)/meshes/visual/J5.dae" scale="1 1 1"/>
 				</geometry>
 			</visual>
@@ -144,5 +144,5 @@
 				<origin rpy="0 0 0" xyz="0 0 0"/>
 				<geometry>
-					<mesh filename="file:///$(find denso_robot_descriptions)/robots/$(arg model)/meshes/J5.dae" scale="1 1 1"/>
+					<mesh filename="file:///$(find denso_robot_descriptions)/robots/$(arg model)/meshes/collision/J5.dae" scale="1 1 1"/>
 				</geometry>
 			</collision>
