Commit message: waypoints on non-cartesian path

File: denso_ros2_ws/src/denso_robot_drivers_ros2/denso_robot_descriptions/robots/vp5243/urdf/denso_robot_joint_limits.xacro (robot description, xacro)
@@ -4,10 +4,10 @@
 		<joint name="$(arg namespace)joint_1">
 			<command_interface name="position">
-				<param name="min">-2.967060</param>
-				<param name="max">2.967060</param>
+				<param name="min">-2.79253</param>
+				<param name="max">2.79253</param>
 			</command_interface>
 			<command_interface name="velocity">
 				<param name="min">0</param>
-				<param name="max">0.392699081698724</param>
+				<param name="max">4.71239</param>
 			</command_interface>
 			<state_interface name="position">
@@ -19,10 +19,10 @@
 		<joint name="$(arg namespace)joint_2">
 			<command_interface name="position">
-				<param name="min">-2.094395</param>
-				<param name="max">2.094395</param>
+				<param name="min">-2.0944</param>
+				<param name="max">2.0944</param>
 			</command_interface>
 			<command_interface name="velocity">
 				<param name="min">0</param>
-				<param name="max">0.261799387799149</param>
+				<param name="max">3.5342917</param>
 			</command_interface>
 			<state_interface name="position">
@@ -34,10 +34,10 @@
 		<joint name="$(arg namespace)joint_3">
 			<command_interface name="position">
-				<param name="min">-2.181662</param>
-				<param name="max">2.705260</param>
+				<param name="min">-2.23402</param>
+				<param name="max">2.37365</param>
 			</command_interface>
 			<command_interface name="velocity">
 				<param name="min">0</param>
-				<param name="max">0.285832571599111</param>
+				<param name="max">4.71239</param>
 			</command_interface>
 			<state_interface name="position">
@@ -49,10 +49,10 @@
 		<joint name="$(arg namespace)joint_4">
 			<command_interface name="position">
-				<param name="min">-2.094395</param>
-				<param name="max">2.094395</param>
+				<param name="min">-2.0944</param>
+				<param name="max">2.0944</param>
 			</command_interface>
 			<command_interface name="velocity">
 				<param name="min">0</param>
-				<param name="max">0.302168853397778</param>
+				<param name="max">5.65487</param>
 			</command_interface>
 			<state_interface name="position">
@@ -69,5 +69,5 @@
 			<command_interface name="velocity">
 				<param name="min">0</param>
-				<param name="max">0.628318530717959</param>
+				<param name="max">5.65487</param>
 			</command_interface>
 			<state_interface name="position">

File: denso_ros2_ws/src/denso_robot_drivers_ros2/denso_robot_descriptions/robots/vp5243/urdf/denso_robot_kinematics.xacro (robot description, xacro)
@@ -50,5 +50,5 @@
 			<origin rpy="0.000000 0.000000 0.000000" xyz="0.000000 0.000000 0.155000"/>
 			<axis xyz="-0.000000 -0.000000 1.000000"/>
-			<limit effort="1" lower="-2.96705972839036" upper="2.96705972839036" velocity="3.73064127613788"/>
+			<limit effort="1" lower="-2.96705972839036" upper="2.96705972839036" velocity="4.71239"/>
 			<dynamics damping="0" friction="0"/>
 		</joint>
@@ -77,5 +77,5 @@
 			<origin rpy="0.000000 0.000000 0.000000" xyz="0.000000 0.000000 0.123500"/>
 			<axis xyz="-0.000000 1.000000 -0.000000"/>
-			<limit effort="1" lower="-2.0943951023932" upper="2.0943951023932" velocity="2.48709418409192"/>
+			<limit effort="1" lower="-2.0943951023932" upper="2.0943951023932" velocity="3.5342917"/>
 			<dynamics damping="0" friction="0"/>
 		</joint>
@@ -104,5 +104,5 @@
 			<origin rpy="0.000000 0.000000 0.000000" xyz="0.000000 0.000000 0.210000"/>
 			<axis xyz="-0.000000 1.000000 -0.000000"/>
-			<limit effort="1" lower="-2.18166156499291" upper="2.70526034059121" velocity="2.71540943019156"/>
+			<limit effort="1" lower="-2.18166156499291" upper="2.70526034059121" velocity="4.71239"/>
 			<dynamics damping="0" friction="0"/>
 		</joint>
@@ -131,5 +131,5 @@
 			<origin rpy="0.000000 0.000000 0.000000" xyz="0.000000 0.000000 0.220000"/>
 			<axis xyz="-0.000000 1.000000 -0.000000"/>
-			<limit effort="1" lower="-2.0943951023932" upper="2.0943951023932" velocity="2.87060410727889"/>
+			<limit effort="1" lower="-2.0943951023932" upper="2.0943951023932" velocity="5.65487"/>
 			<dynamics damping="0" friction="0"/>
 		</joint>
@@ -158,5 +158,5 @@
 			<origin rpy="0.000000 0.000000 0.000000" xyz="0.000000 0.000000 0.070000"/>
 			<axis xyz="-0.000000 -0.000000 1.000000"/>
-			<limit effort="1" lower="-6.28318530717959" upper="6.28318530717959" velocity="5.96902604182061"/>
+			<limit effort="1" lower="-6.28318530717959" upper="6.28318530717959" velocity="5.65487"/>
 			<dynamics damping="0" friction="0"/>
 		</joint>
