Commit message: adding vp5243 with source code from denso

File: denso_ros2_ws/src/denso_robot_drivers_ros2/denso_robot_descriptions/robots/vp5243/urdf/denso_robot.ros2_control.xacro (robot description, xacro)
@@ -2,20 +2,20 @@
 <robot xmlns:xacro="http://www.ros.org/wiki/xacro">
   <xacro:macro name="denso_robot_ros2_control" params="name namespace
-	robot_name
+    robot_name
     sim:=false fake_sensor_commands:=false
     ip_address
     model
-    robot_joints joint_1 joint_2 joint_3 joint_4 joint_5
+    robot_joints joint_1 joint_2 joint_3 joint_4 joint_5 joint_6
     arm_group
     send_format recv_format
-	controller_type
+    controller_type
     verbose
     ">
     <ros2_control name="${namespace}${name}" type="system">
-	<!-- joint limits include -->
-	<xacro:include filename="$(find denso_robot_descriptions)/robots/$(arg model)/urdf/denso_robot_joint_limits.xacro" />
+  <!-- joint limits include -->
+  <xacro:include filename="$(find denso_robot_descriptions)/robots/$(arg model)/urdf/denso_robot_joint_limits.xacro" />
       <hardware>
         <xacro:if value="${sim}">
-      	  <plugin>gazebo_ros2_control/GazeboSystem</plugin>
+          <plugin>gazebo_ros2_control/GazeboSystem</plugin>
         </xacro:if>
         <xacro:unless value="${sim}">
@@ -32,4 +32,5 @@
           <param name="joint_4">${joint_4}</param>
           <param name="joint_5">${joint_5}</param>
+          <param name="joint_6">${joint_6}</param>
           <param name="arm_group">${arm_group}</param>
           <param name="send_format">${send_format}</param>

File: denso_ros2_ws/src/denso_robot_drivers_ros2/denso_robot_descriptions/robots/vp5243/urdf/denso_robot_joint_limits.xacro (robot description, xacro)
@@ -1,80 +1,95 @@
-<?xml version='1.0' encoding='UTF-8'?>
+<?xml version="1.0"?>
 <robot xmlns:xacro="http://www.ros.org/wiki/xacro">
-	<xacro:macro name="denso_robot_control_limits" params="namespace">
-		<joint name="$(arg namespace)joint_1">
-			<command_interface name="position">
-				<param name="min">-2.79253</param>
-				<param name="max">2.79253</param>
-			</command_interface>
-			<command_interface name="velocity">
-				<param name="min">0</param>
-				<param name="max">4.71239</param>
-			</command_interface>
-			<state_interface name="position">
-                <param name="initial_value">0.0</param>
-            </state_interface>
-			<state_interface name="velocity"/>
-			<state_interface name="effort"/>
-		</joint>
-		<joint name="$(arg namespace)joint_2">
-			<command_interface name="position">
-				<param name="min">-2.0944</param>
-				<param name="max">2.0944</param>
-			</command_interface>
-			<command_interface name="velocity">
-				<param name="min">0</param>
-				<param name="max">3.5342917</param>
-			</command_interface>
-			<state_interface name="position">
-                <param name="initial_value">0.0</param>
-            </state_interface>
-			<state_interface name="velocity"/>
-			<state_interface name="effort"/>
-		</joint>
-		<joint name="$(arg namespace)joint_3">
-			<command_interface name="position">
-				<param name="min">-2.23402</param>
-				<param name="max">2.37365</param>
-			</command_interface>
-			<command_interface name="velocity">
-				<param name="min">0</param>
-				<param name="max">4.71239</param>
-			</command_interface>
-			<state_interface name="position">
-                <param name="initial_value">1.57</param>
-            </state_interface>
-			<state_interface name="velocity"/>
-			<state_interface name="effort"/>
-		</joint>
-		<joint name="$(arg namespace)joint_4">
-			<command_interface name="position">
-				<param name="min">-2.0944</param>
-				<param name="max">2.0944</param>
-			</command_interface>
-			<command_interface name="velocity">
-				<param name="min">0</param>
-				<param name="max">5.65487</param>
-			</command_interface>
-			<state_interface name="position">
-                <param name="initial_value">1.57</param>
-            </state_interface>
-			<state_interface name="velocity"/>
-			<state_interface name="effort"/>
-		</joint>
-		<joint name="$(arg namespace)joint_5">
-			<command_interface name="position">
-				<param name="min">-6.283185</param>
-				<param name="max">6.283185</param>
-			</command_interface>
-			<command_interface name="velocity">
-				<param name="min">0</param>
-				<param name="max">5.65487</param>
-			</command_interface>
-			<state_interface name="position">
-                <param name="initial_value">0.0</param>
-            </state_interface>
-			<state_interface name="velocity"/>
-			<state_interface name="effort"/>
-		</joint>
-	</xacro:macro>
+  <xacro:macro name="denso_robot_control_limits" params="namespace">
+    <joint name="$(arg namespace)joint_1">
+      <command_interface name="position">
+        <param name="min">-2.792527</param>
+        <param name="max">2.792527</param>
+      </command_interface>
+      <command_interface name="velocity">
+        <param name="min">0</param>
+        <param name="max">1</param>
+      </command_interface>
+      <state_interface name="position">
+        <param name="initial_value">0.0</param>
+      </state_interface>
+      <state_interface name="velocity"/>
+      <state_interface name="effort"/>
+    </joint>
+    <joint name="$(arg namespace)joint_2">
+      <command_interface name="position">
+        <param name="min">-2.094395</param>
+        <param name="max">2.094395</param>
+      </command_interface>
+      <command_interface name="velocity">
+        <param name="min">0</param>
+        <param name="max">1</param>
+      </command_interface>
+      <state_interface name="position">
+        <param name="initial_value">0.0</param>
+      </state_interface>
+      <state_interface name="velocity"/>
+      <state_interface name="effort"/>
+    </joint>
+    <joint name="$(arg namespace)joint_3">
+      <command_interface name="position">
+        <param name="min">-2.234021</param>
+        <param name="max">2.373648</param>
+      </command_interface>
+      <command_interface name="velocity">
+        <param name="min">0</param>
+        <param name="max">1</param>
+      </command_interface>
+      <state_interface name="position">
+        <param name="initial_value">1.57</param>
+      </state_interface>
+      <state_interface name="velocity"/>
+      <state_interface name="effort"/>
+    </joint>
+    <joint name="$(arg namespace)joint_4">
+      <command_interface name="position">
+        <param name="min">-2.792527</param>
+        <param name="max">2.792527</param>
+      </command_interface>
+      <command_interface name="velocity">
+        <param name="min">0</param>
+        <param name="max">1</param>
+      </command_interface>
+      <state_interface name="position">
+        <param name="initial_value">0.0</param>
+      </state_interface>
+      <state_interface name="velocity"/>
+      <state_interface name="effort"/>
+    </joint>
+    <joint name="$(arg namespace)joint_5">
+      <command_interface name="position">
+        <param name="min">-2.094395</param>
+        <param name="max">2.094395</param>
+      </command_interface>
+      <command_interface name="velocity">
+        <param name="min">0</param>
+        <param name="max">1</param>
+      </command_interface>
+      <state_interface name="position">
+        <param name="initial_value">1.57</param>
+      </state_interface>
+      <state_interface name="velocity"/>
+      <state_interface name="effort"/>
+    </joint>
+    <joint name="$(arg namespace)joint_6">
+      <command_interface name="position">
+        <param name="min">-6.283185</param>
+        <param name="max">6.283185</param>
+      </command_interface>
+      <command_interface name="velocity">
+        <param name="min">0</param>
+        <param name="max">1</param>
+      </command_interface>
+      <state_interface name="position">
+        <param name="initial_value">0.0</param>
+      </state_interface>
+      <state_interface name="velocity"/>
+      <state_interface name="effort"/>
+    </joint>
+  </xacro:macro>
 </robot>

File: denso_ros2_ws/src/denso_robot_drivers_ros2/denso_robot_descriptions/robots/vp5243/urdf/denso_robot_kinematics.xacro (robot description, xacro)
@@ -1,164 +1,191 @@
-<?xml version='1.0' encoding='UTF-8'?>
+<?xml version="1.0"?>
 <robot xmlns:xacro="http://www.ros.org/wiki/xacro">
-	<xacro:macro name="denso_robot_arm_kinematics" params="namespace model">
-		<link name="world"/>
-		<joint name="$(arg namespace)joint_w" type="fixed">
-			<parent link="world"/>
-			<child link="$(arg namespace)base_link"/>
-		</joint>
-		<link name="$(arg namespace)base_link">
-			<visual>
-				<origin rpy="0 0 0" xyz="0 0 0"/>
-				<geometry>
-					<mesh filename="file:///$(find denso_robot_descriptions)/robots/$(arg model)/meshes/visual/base_link.dae" scale="1 1 1"/>
-				</geometry>
-			</visual>
-			<collision>
-				<origin rpy="0 0 0" xyz="0 0 0"/>
-				<geometry>
-					<mesh filename="file:///$(find denso_robot_descriptions)/robots/$(arg model)/meshes/collision/base_link.dae" scale="1 1 1"/>
-				</geometry>
-			</collision>
-			<inertial>
-				<mass value="1"/>
-				<origin rpy="0.000000 0.000000 0.000000" xyz="0.000000 0.000000 0.000000"/>
-				<inertia ixx="1" ixy="0" ixz="0" iyy="1" iyz="0" izz="1"/>
-			</inertial>
-		</link>
-		<link name="$(arg namespace)J1">
-			<visual>
-				<origin rpy="0 0 0" xyz="0 0 0"/>
-				<geometry>
-					<mesh filename="file:///$(find denso_robot_descriptions)/robots/$(arg model)/meshes/visual/J1.dae" scale="1 1 1"/>
-				</geometry>
-			</visual>
-			<collision>
-				<origin rpy="0 0 0" xyz="0 0 0"/>
-				<geometry>
-					<mesh filename="file:///$(find denso_robot_descriptions)/robots/$(arg model)/meshes/collision/J1.dae" scale="1 1 1"/>
-				</geometry>
-			</collision>
-			<inertial>
-				<mass value="1"/>
-				<origin rpy="0.000000 0.000000 0.000000" xyz="0.000000 0.000000 0.000000"/>
-				<inertia ixx="1" ixy="0" ixz="0" iyy="1" iyz="0" izz="1"/>
-			</inertial>
-		</link>
-		<joint name="$(arg namespace)joint_1" type="revolute">
-			<parent link="$(arg namespace)base_link"/>
-			<child link="$(arg namespace)J1"/>
-			<origin rpy="0.000000 0.000000 0.000000" xyz="0.000000 0.000000 0.155000"/>
-			<axis xyz="-0.000000 -0.000000 1.000000"/>
-			<limit effort="1" lower="-2.96705972839036" upper="2.96705972839036" velocity="4.71239"/>
-			<dynamics damping="0" friction="0"/>
-		</joint>
-		<link name="$(arg namespace)J2">
-			<visual>
-				<origin rpy="0 0 0" xyz="0 0 0"/>
-				<geometry>
-					<mesh filename="file:///$(find denso_robot_descriptions)/robots/$(arg model)/meshes/visual/J2.dae" scale="1 1 1"/>
-				</geometry>
-			</visual>
-			<collision>
-				<origin rpy="0 0 0" xyz="0 0 0"/>
-				<geometry>
-					<mesh filename="file:///$(find denso_robot_descriptions)/robots/$(arg model)/meshes/collision/J2.dae" scale="1 1 1"/>
-				</geometry>
-			</collision>
-			<inertial>
-				<mass value="1"/>
-				<origin rpy="0.000000 0.000000 0.000000" xyz="0.000000 0.000000 0.000000"/>
-				<inertia ixx="1" ixy="0" ixz="0" iyy="1" iyz="0" izz="1"/>
-			</inertial>
-		</link>
-		<joint name="$(arg namespace)joint_2" type="revolute">
-			<parent link="$(arg namespace)J1"/>
-			<child link="$(arg namespace)J2"/>
-			<origin rpy="0.000000 0.000000 0.000000" xyz="0.000000 0.000000 0.123500"/>
-			<axis xyz="-0.000000 1.000000 -0.000000"/>
-			<limit effort="1" lower="-2.0943951023932" upper="2.0943951023932" velocity="3.5342917"/>
-			<dynamics damping="0" friction="0"/>
-		</joint>
-		<link name="$(arg namespace)J3">
-			<visual>
-				<origin rpy="0 0 0" xyz="0 0 0"/>
-				<geometry>
-					<mesh filename="file:///$(find denso_robot_descriptions)/robots/$(arg model)/meshes/visual/J3.dae" scale="1 1 1"/>
-				</geometry>
-			</visual>
-			<collision>
-				<origin rpy="0 0 0" xyz="0 0 0"/>
-				<geometry>
-					<mesh filename="file:///$(find denso_robot_descriptions)/robots/$(arg model)/meshes/collision/J3.dae" scale="1 1 1"/>
-				</geometry>
-			</collision>
-			<inertial>
-				<mass value="1"/>
-				<origin rpy="0.000000 0.000000 0.000000" xyz="0.000000 0.000000 0.000000"/>
-				<inertia ixx="1" ixy="0" ixz="0" iyy="1" iyz="0" izz="1"/>
-			</inertial>
-		</link>
-		<joint name="$(arg namespace)joint_3" type="revolute">
-			<parent link="$(arg namespace)J2"/>
-			<child link="$(arg namespace)J3"/>
-			<origin rpy="0.000000 0.000000 0.000000" xyz="0.000000 0.000000 0.210000"/>
-			<axis xyz="-0.000000 1.000000 -0.000000"/>
-			<limit effort="1" lower="-2.18166156499291" upper="2.70526034059121" velocity="4.71239"/>
-			<dynamics damping="0" friction="0"/>
-		</joint>
-		<link name="$(arg namespace)J4">
-			<visual>
-				<origin rpy="0 0 0" xyz="0 0 0"/>
-				<geometry>
-					<mesh filename="file:///$(find denso_robot_descriptions)/robots/$(arg model)/meshes/visual/J4.dae" scale="1 1 1"/>
-				</geometry>
-			</visual>
-			<collision>
-				<origin rpy="0 0 0" xyz="0 0 0"/>
-				<geometry>
-					<mesh filename="file:///$(find denso_robot_descriptions)/robots/$(arg model)/meshes/collision/J4.dae" scale="1 1 1"/>
-				</geometry>
-			</collision>
-			<inertial>
-				<mass value="1"/>
-				<origin rpy="0.000000 0.000000 0.000000" xyz="0.000000 0.000000 0.000000"/>
-				<inertia ixx="1" ixy="0" ixz="0" iyy="1" iyz="0" izz="1"/>
-			</inertial>
-		</link>
-		<joint name="$(arg namespace)joint_4" type="revolute">
-			<parent link="$(arg namespace)J3"/>
-			<child link="$(arg namespace)J4"/>
-			<origin rpy="0.000000 0.000000 0.000000" xyz="0.000000 0.000000 0.220000"/>
-			<axis xyz="-0.000000 1.000000 -0.000000"/>
-			<limit effort="1" lower="-2.0943951023932" upper="2.0943951023932" velocity="5.65487"/>
-			<dynamics damping="0" friction="0"/>
-		</joint>
-		<link name="$(arg namespace)J5">
-			<visual>
-				<origin rpy="0 0 0" xyz="0 0 0"/>
-				<geometry>
-					<mesh filename="file:///$(find denso_robot_descriptions)/robots/$(arg model)/meshes/visual/J5.dae" scale="1 1 1"/>
-				</geometry>
-			</visual>
-			<collision>
-				<origin rpy="0 0 0" xyz="0 0 0"/>
-				<geometry>
-					<mesh filename="file:///$(find denso_robot_descriptions)/robots/$(arg model)/meshes/collision/J5.dae" scale="1 1 1"/>
-				</geometry>
-			</collision>
-			<inertial>
-				<mass value="1"/>
-				<origin rpy="0.000000 0.000000 0.000000" xyz="0.000000 0.000000 0.000000"/>
-				<inertia ixx="1" ixy="0" ixz="0" iyy="1" iyz="0" izz="1"/>
-			</inertial>
-		</link>
-		<joint name="$(arg namespace)joint_5" type="revolute">
-			<parent link="$(arg namespace)J4"/>
-			<child link="$(arg namespace)J5"/>
-			<origin rpy="0.000000 0.000000 0.000000" xyz="0.000000 0.000000 0.070000"/>
-			<axis xyz="-0.000000 -0.000000 1.000000"/>
-			<limit effort="1" lower="-6.28318530717959" upper="6.28318530717959" velocity="5.65487"/>
-			<dynamics damping="0" friction="0"/>
-		</joint>
-	</xacro:macro>
+  <xacro:macro name="denso_robot_arm_kinematics" params="namespace model">
+    <link name="world"/>
+    <joint name="$(arg namespace)joint_w" type="fixed">
+      <parent link="world"/>
+      <child link="$(arg namespace)base_link"/>
+    </joint>
+    <link name="$(arg namespace)base_link">
+      <visual>
+        <origin rpy="0 0 0" xyz="0 0 0"/>
+        <geometry>
+          <mesh filename="file:///$(find denso_robot_descriptions)/robots/$(arg model)/meshes/base_link.dae" scale="1 1 1"/>
+        </geometry>
+      </visual>
+      <collision>
+        <origin rpy="0 0 0" xyz="0 0 0"/>
+        <geometry>
+          <mesh filename="file:///$(find denso_robot_descriptions)/robots/$(arg model)/meshes/base_link.dae" scale="1 1 1"/>
+        </geometry>
+      </collision>
+      <inertial>
+        <mass value="1"/>
+        <origin rpy="0.000000 0.000000 0.000000" xyz="0.000000 0.000000 0.000000"/>
+        <inertia ixx="1" ixy="0" ixz="0" iyy="1" iyz="0" izz="1"/>
+      </inertial>
+    </link>
+    <link name="$(arg namespace)J1">
+      <visual>
+        <origin rpy="0 0 0" xyz="0 0 0"/>
+        <geometry>
+          <mesh filename="file:///$(find denso_robot_descriptions)/robots/$(arg model)/meshes/J1.dae" scale="1 1 1"/>
+        </geometry>
+      </visual>
+      <collision>
+        <origin rpy="0 0 0" xyz="0 0 0"/>
+        <geometry>
+          <mesh filename="file:///$(find denso_robot_descriptions)/robots/$(arg model)/meshes/J1.dae" scale="1 1 1"/>
+        </geometry>
+      </collision>
+      <inertial>
+        <mass value="1"/>
+        <origin rpy="0.000000 0.000000 0.000000" xyz="0.000000 0.000000 0.000000"/>
+        <inertia ixx="1" ixy="0" ixz="0" iyy="1" iyz="0" izz="1"/>
+      </inertial>
+    </link>
+    <joint name="$(arg namespace)joint_1" type="revolute">
+      <parent link="$(arg namespace)base_link"/>
+      <child link="$(arg namespace)J1"/>
+      <origin rpy="0.000000 0.000000 0.000000" xyz="0.000000 0.000000 0.000000"/>
+      <axis xyz="-0.000000 -0.000000 1.000000"/>
+      <limit effort="1" lower="-2.79252680319093" upper="2.79252680319093" velocity="1"/>
+      <dynamics damping="0" friction="0"/>
+    </joint>
+    <link name="$(arg namespace)J2">
+      <visual>
+        <origin rpy="0 0 0" xyz="0 0 0"/>
+        <geometry>
+          <mesh filename="file:///$(find denso_robot_descriptions)/robots/$(arg model)/meshes/J2.dae" scale="1 1 1"/>
+        </geometry>
+      </visual>
+      <collision>
+        <origin rpy="0 0 0" xyz="0 0 0"/>
+        <geometry>
+          <mesh filename="file:///$(find denso_robot_descriptions)/robots/$(arg model)/meshes/J2.dae" scale="1 1 1"/>
+        </geometry>
+      </collision>
+      <inertial>
+        <mass value="1"/>
+        <origin rpy="0.000000 0.000000 0.000000" xyz="0.000000 0.000000 0.000000"/>
+        <inertia ixx="1" ixy="0" ixz="0" iyy="1" iyz="0" izz="1"/>
+      </inertial>
+    </link>
+    <joint name="$(arg namespace)joint_2" type="revolute">
+      <parent link="$(arg namespace)J1"/>
+      <child link="$(arg namespace)J2"/>
+      <origin rpy="0.000000 0.000000 0.000000" xyz="0.000000 0.000000 0.280000"/>
+      <axis xyz="-0.000000 1.000000 -0.000000"/>
+      <limit effort="1" lower="-2.0943951023932" upper="2.0943951023932" velocity="1"/>
+      <dynamics damping="0" friction="0"/>
+    </joint>
+    <link name="$(arg namespace)J3">
+      <visual>
+        <origin rpy="0 0 0" xyz="0 0 0"/>
+        <geometry>
+          <mesh filename="file:///$(find denso_robot_descriptions)/robots/$(arg model)/meshes/J3.dae" scale="1 1 1"/>
+        </geometry>
+      </visual>
+      <collision>
+        <origin rpy="0 0 0" xyz="0 0 0"/>
+        <geometry>
+          <mesh filename="file:///$(find denso_robot_descriptions)/robots/$(arg model)/meshes/J3.dae" scale="1 1 1"/>
+        </geometry>
+      </collision>
+      <inertial>
+        <mass value="1"/>
+        <origin rpy="0.000000 0.000000 0.000000" xyz="0.000000 0.000000 0.000000"/>
+        <inertia ixx="1" ixy="0" ixz="0" iyy="1" iyz="0" izz="1"/>
+      </inertial>
+    </link>
+    <joint name="$(arg namespace)joint_3" type="revolute">
+      <parent link="$(arg namespace)J2"/>
+      <child link="$(arg namespace)J3"/>
+      <origin rpy="0.000000 0.000000 0.000000" xyz="0.000000 0.000000 0.210000"/>
+      <axis xyz="-0.000000 1.000000 -0.000000"/>
+      <limit effort="1" lower="-2.23402144255274" upper="2.37364778271229" velocity="1"/>
+      <dynamics damping="0" friction="0"/>
+    </joint>
+    <link name="$(arg namespace)J4">
+      <visual>
+        <origin rpy="0 0 0" xyz="0 0 0"/>
+        <geometry>
+          <!-- <mesh filename="file:///$(find denso_robot_descriptions)/robots/$(arg model)/meshes/J4.dae" scale="1 1 1"/> -->
+        </geometry>
+      </visual>
+      <collision>
+        <origin rpy="0 0 0" xyz="0 0 0"/>
+        <geometry>
+          <!-- <mesh filename="file:///$(find denso_robot_descriptions)/robots/$(arg model)/meshes/J4.dae" scale="1 1 1"/> -->
+        </geometry>
+      </collision>
+      <inertial>
+        <mass value="1"/>
+        <origin rpy="0.000000 0.000000 0.000000" xyz="0.000000 0.000000 0.000000"/>
+        <inertia ixx="1" ixy="0" ixz="0" iyy="1" iyz="0" izz="1"/>
+      </inertial>
+    </link>
+    <joint name="$(arg namespace)joint_4" type="fixed">
+      <parent link="$(arg namespace)J3"/>
+      <child link="$(arg namespace)J4"/>
+      <origin rpy="0.000000 0.000000 0.000000" xyz="0.000000 0.000000 0.000000"/>
+      <axis xyz="-0.000000 -0.000000 -0.000000"/>
+      <limit effort="1" lower="-2.79252680319093" upper="2.79252680319093" velocity="1"/>
+      <dynamics damping="0" friction="0"/>
+    </joint>
+    <link name="$(arg namespace)J5">
+      <visual>
+        <origin rpy="0 0 0" xyz="0 0 0"/>
+        <geometry>
+          <mesh filename="file:///$(find denso_robot_descriptions)/robots/$(arg model)/meshes/J5.dae" scale="1 1 1"/>
+        </geometry>
+      </visual>
+      <collision>
+        <origin rpy="0 0 0" xyz="0 0 0"/>
+        <geometry>
+          <mesh filename="file:///$(find denso_robot_descriptions)/robots/$(arg model)/meshes/J5.dae" scale="1 1 1"/>
+        </geometry>
+      </collision>
+      <inertial>
+        <mass value="1"/>
+        <origin rpy="0.000000 0.000000 0.000000" xyz="0.000000 0.000000 0.000000"/>
+        <inertia ixx="1" ixy="0" ixz="0" iyy="1" iyz="0" izz="1"/>
+      </inertial>
+    </link>
+    <joint name="$(arg namespace)joint_5" type="revolute">
+      <parent link="$(arg namespace)J4"/>
+      <child link="$(arg namespace)J5"/>
+      <origin rpy="0.000000 0.000000 0.000000" xyz="0.000000 0.000000 0.220000"/>
+      <axis xyz="-0.000000 1.000000 -0.000000"/>
+      <limit effort="1" lower="-2.0943951023932" upper="2.0943951023932" velocity="1"/>
+      <dynamics damping="0" friction="0"/>
+    </joint>
+    <link name="$(arg namespace)J6">
+      <visual>
+        <origin rpy="0 0 0" xyz="0 0 0"/>
+        <geometry>
+          <mesh filename="file:///$(find denso_robot_descriptions)/robots/$(arg model)/meshes/J6.dae" scale="1 1 1"/>
+        </geometry>
+      </visual>
+      <collision>
+        <origin rpy="0 0 0" xyz="0 0 0"/>
+        <geometry>
+          <mesh filename="file:///$(find denso_robot_descriptions)/robots/$(arg model)/meshes/J6.dae" scale="1 1 1"/>
+        </geometry>
+      </collision>
+      <inertial>
+        <mass value="1"/>
+        <origin rpy="0.000000 0.000000 0.000000" xyz="0.000000 0.000000 0.000000"/>
+        <inertia ixx="1" ixy="0" ixz="0" iyy="1" iyz="0" izz="1"/>
+      </inertial>
+    </link>
+    <joint name="$(arg namespace)joint_6" type="revolute">
+      <parent link="$(arg namespace)J5"/>
+      <child link="$(arg namespace)J6"/>
+      <origin rpy="0.000000 0.000000 0.000000" xyz="0.000000 0.000000 0.070000"/>
+      <axis xyz="-0.000000 -0.000000 1.000000"/>
+      <limit effort="1" lower="-6.28318530717959" upper="6.28318530717959" velocity="1"/>
+      <dynamics damping="0" friction="0"/>
+    </joint>
+  </xacro:macro>
 </robot>
