Commit message: adding vp5243 with source code from denso

File: denso_ros2_ws/src/denso_robot_drivers_ros2/denso_robot_descriptions/robots/vp5243/urdf/denso_robot_macro.xacro (robot description, xacro)
@@ -21,11 +21,12 @@
     <!-- Robot data required by the denso driver -->
     <xacro:arg name="ip_address" default="192.168.0.1"/>
-    <xacro:arg name="robot_name" default="VP-5243M"/> <!-- "robot_name" param must be consistent with the @TYPE_NAME variable of the real robot !! -->
+    <xacro:arg name="robot_name" default="VP-5243"/> <!-- "robot_name" param must be consistent with the @TYPE_NAME variable of the real robot !! -->
     <xacro:arg name="robot_joints" default="6"/> <!-- number of total joints in the kinematic chain -->
     <xacro:arg name="joint_1" default="1"/> <!-- 0 = prismatic , 1 = revolute -->
     <xacro:arg name="joint_2" default="1"/> <!-- 0 = prismatic , 1 = revolute -->
     <xacro:arg name="joint_3" default="1"/> <!-- 0 = prismatic , 1 = revolute -->
-    <xacro:arg name="joint_4" default="1"/> <!-- 0 = prismatic , 1 = revolute -->
+    <xacro:arg name="joint_4" default="-1"/> <!-- 0 = prismatic , 1 = revolute -->
     <xacro:arg name="joint_5" default="1"/> <!-- 0 = prismatic , 1 = revolute -->
+    <xacro:arg name="joint_6" default="1"/> <!-- 0 = prismatic , 1 = revolute -->
     <xacro:arg name="controller_type" default="8"/> <!-- 8 = RC8 , 9 = RC9 -->
     <xacro:arg name="arm_group" default="0"/>
@@ -51,4 +52,5 @@
       joint_4="$(arg joint_4)"
       joint_5="$(arg joint_5)"
+      joint_6="$(arg joint_6)"
       arm_group="$(arg arm_group)"
       controller_type="$(arg controller_type)"
@@ -62,8 +64,8 @@
     <xacro:denso_robot_arm_kinematics namespace="$(arg namespace)" model="$(arg model)" />
     <gazebo>
-	    <plugin filename="libgazebo_ros2_control.so" name="gazebo_ros2_control">
-      		<parameters>$(find denso_robot_moveit_config)/robots/$(arg model)/config/denso_robot_controllers.yaml</parameters>
-    	</plugin>
-  	</gazebo>
+      <plugin filename="libgazebo_ros2_control.so" name="gazebo_ros2_control">
+        <parameters>$(find denso_robot_moveit_config)/robots/$(arg model)/config/denso_robot_controllers.yaml</parameters>
+      </plugin>
+    </gazebo>
   </xacro:macro>
 </robot>

File: denso_ros2_ws/src/denso_robot_drivers_ros2/denso_robot_descriptions/robots/vp5243/urdf/denso_robot_transmissions.xacro (robot description, xacro)
@@ -52,4 +52,13 @@
       </actuator>
     </transmission>
+    <transmission name="${namespace}trans_6">
+      <type>transmission_interface/SimpleTransmission</type>
+      <joint name="${namespace}joint_6">
+        <hardwareInterface>${hw_interface}</hardwareInterface>
+      </joint>
+      <actuator name="${namespace}motor_6">
+        <mechanicalReduction>1</mechanicalReduction>
+      </actuator>
+    </transmission>
   </xacro:macro>
 </robot>

File: denso_ros2_ws/src/denso_robot_drivers_ros2/denso_robot_descriptions/urdf/denso_robot.urdf.xacro (robot description, xacro)
@@ -30,5 +30,5 @@
    </xacro:if>
    <xacro:if value="${'$(arg model)' == 'vp5243'}">
-     <xacro:property name="tool_parent_link" value="$(arg namespace)J5" />
+     <xacro:property name="tool_parent_link" value="$(arg namespace)J6" />
    </xacro:if>
    <xacro:unless value="${'$(arg tool)' == 'none'}">

File: denso_ros2_ws/src/denso_robot_drivers_ros2/denso_robot_moveit_config/robots/vp5243/srdf/denso_robot_macro.srdf.xacro (robot description, xacro)
@@ -1,22 +1,44 @@
 <?xml version="1.0" encoding="UTF-8"?>
 <robot xmlns:xacro="http://wiki.ros.org/xacro">
+<!--This does not replace URDF, and is not an extension of URDF.
+    This is a format for representing semantic information about the robot structure.
+    A URDF file must exist for this robot as well, where the joints and the links that are referenced are defined
+-->
   <xacro:macro name="denso_robot_srdf" params="name namespace tool">
-    <group name="arm">
-      <xacro:if value="${tool == 'none'}">
-        <chain base_link="$(arg namespace)base_link" tip_link="$(arg namespace)J5"/>
-      </xacro:if>
-      <xacro:if value="${tool != 'none'}">
-        <chain base_link="$(arg namespace)base_link" tip_link="$(arg namespace)tool_link"/>
-      </xacro:if>
-    </group>
+    <!--GROUPS - Representation of a set of joints and links. This can be useful for specifying DOF to plan for, defining arms, end effectors, etc-->
+    <!--LINKS - When a link is specified, the parent joint of that link (if it exists) is automatically included-->
+    <!--JOINTS - When a joint is specified, the child link of that joint (which will always exist) is automatically included-->
+    <!--CHAINS - When a chain is specified, all the links along the chain (including endpoints) are included in the group. Additionally, all the joints that are parents to included links are also included. This means that joints along the chain and the parent joint of the base link are included in the group-->
+    <!--SUBGROUPS - Groups can also be formed by referencing to already defined group names-->
+    <group name="${namespace}arm">
+		<joint name="$(arg namespace)joint_1"/>
+		<joint name="$(arg namespace)joint_2"/>
+		<joint name="$(arg namespace)joint_3"/>
+		<joint name="$(arg namespace)joint_4"/>
+		<joint name="$(arg namespace)joint_5"/>
+		<joint name="$(arg namespace)joint_6"/>
+    <xacro:if value="${tool == 'none'}">
+      <chain base_link="$(arg namespace)base_link" tip_link="$(arg namespace)J6"/>
+    </xacro:if>
+    <xacro:if value="${tool != 'none'}">
+      <chain base_link="$(arg namespace)base_link" tip_link="$(arg namespace)tool_link"/>
+    </xacro:if>
+	</group>
+    <!--GROUP STATES - Purpose - Define a named state for a particular group, in terms of joint values. This is useful to define states like 'folded arms'-->
+    <!--END EFFECTOR - Purpose - Represent information about an end effector.-->
+    <!--VIRTUAL JOINT - Purpose - this element defines a virtual joint between a robot link and an external frame of reference (considered fixed with respect to the robot)-->
     <virtual_joint name="${namespace}fixed_base" type="fixed" parent_frame="world" child_link="${namespace}base_link" />
-    <disable_collisions link1="$(arg namespace)J1" link2="$(arg namespace)base_link" reason="Adjacent"/>
-    <disable_collisions link1="$(arg namespace)J1" link2="$(arg namespace)J2" reason="Adjacent"/>
-    <disable_collisions link1="$(arg namespace)J2" link2="$(arg namespace)J3" reason="Adjacent"/>
-    <disable_collisions link1="$(arg namespace)J3" link2="$(arg namespace)J4" reason="Adjacent"/>
-    <disable_collisions link1="$(arg namespace)J4" link2="$(arg namespace)J5" reason="Adjacent"/>
-    <xacro:if value="${tool != 'none'}">
-      <disable_collisions link1="$(arg namespace)J5" link2="$(arg namespace)tool_link" reason="Attached by fixed joint" />
-    </xacro:if>
+    <!--DISABLE COLLISIONS - By default it is assumed that any link of the robot could potentially come into collision with any other link in the robot. This tag disables collision checking between a specified pair of links. -->
+	<disable_collisions link1="$(arg namespace)J6" link2="$(arg namespace)J3" reason="Never"/>
+	<disable_collisions link1="$(arg namespace)J6" link2="$(arg namespace)J5" reason="Adjacent"/>
+	<disable_collisions link1="$(arg namespace)J1" link2="$(arg namespace)J2" reason="Adjacent"/>
+	<disable_collisions link1="$(arg namespace)J1" link2="$(arg namespace)base_link" reason="Adjacent"/>
+	<disable_collisions link1="$(arg namespace)J2" link2="$(arg namespace)J3" reason="Adjacent"/>
+	<disable_collisions link1="$(arg namespace)J3" link2="$(arg namespace)J4" reason="Adjacent"/>
+	<disable_collisions link1="$(arg namespace)J3" link2="$(arg namespace)J5" reason="Never"/>
+	<disable_collisions link1="$(arg namespace)J4" link2="$(arg namespace)J5" reason="Adjacent"/>
+  <xacro:if value="${tool != 'none'}">
+      <disable_collisions link1="$(arg namespace)J6" link2="$(arg namespace)tool_link" reason="Attached by fixed joint" />
+  </xacro:if>
   </xacro:macro>
 </robot>
