Commit message: attempting to refactor staubli ros package, not working at this point

File: denso_ros2_ws/src/Staubli_ROS2-humble/staubli_robot_description/urdf/common_materials.xacro (robot description, xacro)
@@ -1,5 +1,5 @@
 <?xml version="1.0"?>
 <robot xmlns:xacro="http://wiki.ros.org/xacro">
-  <xacro:include filename="$(find staubli_tx2_60l_description)/urdf/common_colours.xacro"/>
+  <xacro:include filename="$(find staubli_robot_description)/urdf/common_colours.xacro"/>
   <!-- default colors for robots -->
   <xacro:macro name="material_staubli_ral_melon_yellow">

File: denso_ros2_ws/src/Staubli_ROS2-humble/staubli_robot_description/urdf/tx2_60l/tx2_60l.xacro (robot description, xacro)
@@ -1,5 +1,5 @@
 <?xml version="1.0" ?>
 <robot name="staubli_tx2_60l" xmlns:xacro="http://wiki.ros.org/xacro">
-  <xacro:include filename="$(find staubli_tx2_60l_description)/urdf/tx2_60l_macro.xacro"/>
+  <xacro:include filename="$(find staubli_robot_description)/urdf/tx2_60l/tx2_60l_macro.xacro"/>
   <xacro:staubli_tx2_60l prefix=""/>
 </robot>

File: denso_ros2_ws/src/Staubli_ROS2-humble/staubli_robot_description/urdf/tx2_60l/tx2_60l_macro.xacro (robot description, xacro)
@@ -1,5 +1,5 @@
 <?xml version="1.0"?>
 <robot xmlns:xacro="http://wiki.ros.org/xacro">
-  <xacro:include filename="$(find staubli_tx2_60l_description)/urdf/common_materials.xacro"/>
+  <xacro:include filename="$(find staubli_robot_description)/urdf/common_materials.xacro"/>
   <xacro:macro name="staubli_tx2_60l" params="prefix">
     <!-- links: main serial chain -->
@@ -8,5 +8,5 @@
         <origin xyz="0 0 0" rpy="0 0 0"/>
         <geometry>
-          <mesh filename="package://staubli_tx2_60l_description/meshes/visual/base_link.stl"/>
+          <mesh filename="package://staubli_robot_description/meshes/tx2_60l/visual/base_link.stl"/>
         </geometry>
         <xacro:material_staubli_ral_melon_yellow />
@@ -15,5 +15,5 @@
         <origin xyz="0 0 0" rpy="0 0 0"/>
         <geometry>
-          <mesh filename="package://staubli_tx2_60l_description/meshes/collision/base_link.stl"/>
+          <mesh filename="package://staubli_robot_description/meshes/tx2_60l/collision/base_link.stl"/>
         </geometry>
       </collision>
@@ -23,5 +23,5 @@
         <origin xyz="0 0 0" rpy="0 0 0"/>
         <geometry>
-          <mesh filename="package://staubli_tx2_60l_description/meshes/visual/link_1.stl"/>
+          <mesh filename="package://staubli_robot_description/meshes/tx2_60l/visual/link_1.stl"/>
         </geometry>
         <xacro:material_staubli_ral_melon_yellow />
@@ -30,5 +30,5 @@
         <origin xyz="0 0 0" rpy="0 0 0"/>
         <geometry>
-          <mesh filename="package://staubli_tx2_60l_description/meshes/collision/link_1.stl"/>
+          <mesh filename="package://staubli_robot_description/meshes/tx2_60l/collision/link_1.stl"/>
         </geometry>
       </collision>
@@ -38,5 +38,5 @@
         <origin xyz="0 0 0" rpy="0 0 0"/>
         <geometry>
-          <mesh filename="package://staubli_tx2_60l_description/meshes/visual/link_2.stl"/>
+          <mesh filename="package://staubli_robot_description/meshes/tx2_60l/visual/link_2.stl"/>
         </geometry>
         <xacro:material_staubli_ral_melon_yellow />
@@ -45,5 +45,5 @@
         <origin xyz="0 0 0" rpy="0 0 0"/>
         <geometry>
-          <mesh filename="package://staubli_tx2_60l_description/meshes/collision/link_2.stl"/>
+          <mesh filename="package://staubli_robot_description/meshes/tx2_60l/collision/link_2.stl"/>
         </geometry>
       </collision>
@@ -53,5 +53,5 @@
         <origin xyz="0 0 0" rpy="0 0 0"/>
         <geometry>
-          <mesh filename="package://staubli_tx2_60l_description/meshes/visual/link_3.stl"/>
+          <mesh filename="package://staubli_robot_description/meshes/tx2_60l/visual/link_3.stl"/>
         </geometry>
         <xacro:material_staubli_ral_melon_yellow />
@@ -60,5 +60,5 @@
         <origin xyz="0 0 0" rpy="0 0 0"/>
         <geometry>
-          <mesh filename="package://staubli_tx2_60l_description/meshes/collision/link_3.stl"/>
+          <mesh filename="package://staubli_robot_description/meshes/tx2_60l/collision/link_3.stl"/>
         </geometry>
       </collision>
@@ -68,5 +68,5 @@
         <origin xyz="0 0 0" rpy="0 0 0"/>
         <geometry>
-          <mesh filename="package://staubli_tx2_60l_description/meshes/visual/link_4.stl"/>
+          <mesh filename="package://staubli_robot_description/meshes/tx2_60l/visual/link_4.stl"/>
         </geometry>
         <xacro:material_staubli_ral_melon_yellow />
@@ -75,5 +75,5 @@
         <origin xyz="0 0 0" rpy="0 0 0"/>
         <geometry>
-          <mesh filename="package://staubli_tx2_60l_description/meshes/collision/link_4.stl"/>
+          <mesh filename="package://staubli_robot_description/meshes/tx2_60l/collision/link_4.stl"/>
         </geometry>
       </collision>
@@ -83,5 +83,5 @@
         <origin xyz="0 0 0" rpy="0 0 0"/>
         <geometry>
-          <mesh filename="package://staubli_tx2_60l_description/meshes/visual/link_5.stl"/>
+          <mesh filename="package://staubli_robot_description/meshes/tx2_60l/visual/link_5.stl"/>
         </geometry>
         <xacro:material_staubli_ral_grey_aluminium />
@@ -90,5 +90,5 @@
         <origin xyz="0 0 0" rpy="0 0 0"/>
         <geometry>
-          <mesh filename="package://staubli_tx2_60l_description/meshes/collision/link_5.stl"/>
+          <mesh filename="package://staubli_robot_description/meshes/tx2_60l/collision/link_5.stl"/>
         </geometry>
       </collision>
@@ -98,5 +98,5 @@
         <origin xyz="0 0 0" rpy="0 0 0"/>
         <geometry>
-          <mesh filename="package://staubli_tx2_60l_description/meshes/visual/link_6.stl"/>
+          <mesh filename="package://staubli_robot_description/meshes/tx2_60l/visual/link_6.stl"/>
         </geometry>
         <xacro:material_staubli_ral_grey_aluminium />
@@ -105,5 +105,5 @@
         <origin xyz="0 0 0" rpy="0 0 0"/>
         <geometry>
-          <mesh filename="package://staubli_tx2_60l_description/meshes/collision/link_6.stl"/>
+          <mesh filename="package://staubli_robot_description/meshes/tx2_60l/collision/link_6.stl"/>
         </geometry>
       </collision>

File: denso_ros2_ws/src/Staubli_ROS2-humble/staubli_robot_moveit_config/config/tx2_60l/staubli_tx2_60l.urdf.xacro (robot description, xacro)
@@ -3,5 +3,5 @@
     <xacro:arg name="initial_positions_file" default="initial_positions.yaml" />
     <!-- Import panda urdf file -->
-    <xacro:include filename="$(find staubli_tx2_60l_description)/urdf/tx2_60l.xacro" />
+    <xacro:include filename="$(find staubli_robot_description)/urdf/tx2_60l/tx2_60l.xacro" />
     <!-- Import staubli ros2_control description -->
     <xacro:include filename="staubli_tx2_60l.ros2_control.xacro" />
