Commit message: gazebo not working with launch

File: denso_ros2_ws/src/Staubli_ROS2-humble/staubli_tx2_60l_description/urdf/common_colours.xacro (robot description, xacro)
@@ -1,18 +1,9 @@
 <?xml version="1.0"?>
 <robot xmlns:xacro="http://wiki.ros.org/xacro">
-  <!-- colours based on RAL values supplied by Staubli -->
-  <!-- all RAL colours converted using http://www.visual-graphics.de/en/customer-care/ral-colours -->
-  <!-- default colours for robots -->
-  <!-- RAL 1028 - Melon yellow - scara (non-textured) and 6-axis (textured) robots -->
   <xacro:property name="colour_staubli_ral_melon_yellow"   value="${255/255} ${155/255} ${  0/255} 1.0" />
-  <!-- RAL 7035 - Light grey - scara robot ESD -->
   <xacro:property name="colour_staubli_ral_light_grey"     value="${197/255} ${199/255} ${196/255} 1.0" />
-  <!-- RAL 7045 - Telegrey 1 - scara robot base (textured) -->
   <xacro:property name="colour_staubli_ral_telegrey_1"     value="${141/255} ${146/255} ${149/255} 1.0" />
-  <!-- RAL 7047 - Telegrey 4 - paint (smooth) -->
   <xacro:property name="colour_staubli_ral_telegrey_4"     value="${200/255} ${200/255} ${199/255} 1.0" />
-  <!-- RAL 9007 - Grey aluminium - HE (smooth) -->
   <xacro:property name="colour_staubli_ral_grey_aluminium" value="${135/255} ${133/255} ${129/255} 1.0" />
-  <!-- RAL 9016 - Traffic white - CR (smooth) -->
   <xacro:property name="colour_staubli_ral_traffic_white"  value="${241/255} ${240/255} ${234/255} 1.0" />
 </robot>

File: denso_ros2_ws/src/Staubli_ROS2-humble/staubli_tx2_60l_moveit_config/config/staubli_tx2_60l.ros2_control.xacro (robot description, xacro)
@@ -1,9 +1,14 @@
 <?xml version="1.0"?>
 <robot xmlns:xacro="http://www.ros.org/wiki/xacro">
-    <xacro:macro name="staubli_tx2_60l_ros2_control" params="name initial_positions_file">
-        <xacro:property name="initial_positions" value="${load_yaml(initial_positions_file)['initial_positions']}"/>
+    <xacro:macro name="staubli_tx2_60l_ros2_control" params="name initial_positions_file sim">
+        <xacro:property name="initial_positions" value="${xacro.load_yaml(initial_positions_file)['initial_positions']}"/>
         <ros2_control name="${name}" type="system">
             <hardware>
-                <plugin>fake_components/GenericSystem</plugin>
+                <xacro:if value="${sim}">
+                    <plugin>gazebo_ros2_control/GazeboSystem</plugin>
+                </xacro:if>
+                <xacro:unless value="${sim}">
+                    <plugin>fake_components/GenericSystem</plugin>
+                </xacro:unless>
             </hardware>
             <joint name="joint_1">

File: denso_ros2_ws/src/Staubli_ROS2-humble/staubli_tx2_60l_moveit_config/config/staubli_tx2_60l.srdf.xacro (robot description, xacro)
@@ -4,5 +4,5 @@
     A URDF file must exist for this robot as well, where the joints and the links that are referenced are defined
 -->
-<robot name="staubli_tx2_60l">
+<robot xmlns:xacro="http://www.ros.org/wiki/xacro" name="staubli_tx2_60l">
     <!--GROUPS: Representation of a set of joints and links. This can be useful for specifying DOF to plan for, defining arms, end effectors, etc-->
     <!--LINKS: When a link is specified, the parent joint of that link (if it exists) is automatically included-->
@@ -10,4 +10,8 @@
     <!--CHAINS: When a chain is specified, all the links along the chain (including endpoints) are included in the group. Additionally, all the joints that are parents to included links are also included. This means that joints along the chain and the parent joint of the base link are included in the group-->
     <!--SUBGROUPS: Groups can also be formed by referencing to already defined group names-->
+    <xacro:arg name="model" default="tx2_60l"/>
+    <xacro:arg name="sim" default="true"/>
+    <xacro:arg name="tool" default="none"/>
+    <xacro:arg name="namespace" default=""/>
     <group name="manipulator">
         <chain base_link="base_link" tip_link="tool0"/>

File: denso_ros2_ws/src/Staubli_ROS2-humble/staubli_tx2_60l_moveit_config/config/staubli_tx2_60l.urdf.xacro (robot description, xacro)
@@ -1,9 +1,27 @@
 <?xml version="1.0"?>
-<robot xmlns:xacro="http://www.ros.org/wiki/xacro" name="staubli">
+<robot xmlns:xacro="http://www.ros.org/wiki/xacro" name="staubli_tx2_60l">
     <xacro:arg name="initial_positions_file" default="initial_positions.yaml" />
-    <!-- Import panda urdf file -->
+    <xacro:arg name="model" default="tx2_60l"/>
+    <xacro:arg name="sim" default="true"/>
+    <xacro:arg name="tool" default="none"/>
+    <xacro:arg name="namespace" default=""/>
+    <xacro:arg name="robot_description_file" default=""/>
     <xacro:include filename="$(find staubli_tx2_60l_description)/urdf/tx2_60l.xacro" />
-    <!-- Import staubli ros2_control description -->
     <xacro:include filename="staubli_tx2_60l.ros2_control.xacro" />
-    <xacro:staubli_tx2_60l_ros2_control name="StaubliTX260lFakeSystem" initial_positions_file="$(arg initial_positions_file)"/>
+    <xacro:staubli_tx2_60l_ros2_control
+        name="StaubliTX260lSystem"
+        initial_positions_file="$(arg initial_positions_file)"
+        sim="$(arg sim)"/>
+    <xacro:if value="$(arg sim)">
+        <gazebo>
+            <plugin filename="libgazebo_ros2_control.so" name="gazebo_ros2_control">
+                <parameters>$(find staubli_tx2_60l_moveit_config)/config/ros2_controllers.yaml</parameters>
+                <robot_param>robot_description</robot_param>
+                <robot_param_node>robot_state_publisher</robot_param_node>
+                <parameters>
+                  robot_description: "$(arg robot_description_file)"
+                </parameters>
+            </plugin>
+        </gazebo>
+    </xacro:if>
 </robot>
