Commit message: not working

File: denso_ros2_ws/src/Staubli_ROS2-humble/staubli_tx2_60l_description/urdf/tx2_60l_macro.xacro (robot description, xacro)
@@ -3,4 +3,12 @@
   <xacro:include filename="$(find staubli_tx2_60l_description)/urdf/common_materials.xacro"/>
   <xacro:macro name="staubli_tx2_60l" params="prefix">
+    <!-- World link - always present so Gazebo Classic SDF conversion gets a proper root.
+         Without this, the URDF->SDF conversion fails with FrameAttachedToGraph errors
+         and gazebo_ros2_control skips all joint interfaces. -->
+    <link name="world"/>
+    <joint name="${prefix}world_joint" type="fixed">
+      <parent link="world"/>
+      <child link="${prefix}base_link"/>
+    </joint>
     <!-- links: main serial chain -->
     <link name="${prefix}base_link">
@@ -18,4 +26,9 @@
         </geometry>
       </collision>
+      <inertial>
+        <mass value="1"/>
+        <origin xyz="0 0 0" rpy="0 0 0"/>
+        <inertia ixx="1" ixy="0" ixz="0" iyy="1" iyz="0" izz="1"/>
+      </inertial>
     </link>
     <link name="${prefix}link_1">
@@ -33,4 +46,9 @@
         </geometry>
       </collision>
+      <inertial>
+        <mass value="1"/>
+        <origin xyz="0 0 0" rpy="0 0 0"/>
+        <inertia ixx="1" ixy="0" ixz="0" iyy="1" iyz="0" izz="1"/>
+      </inertial>
     </link>
     <link name="${prefix}link_2">
@@ -48,4 +66,9 @@
         </geometry>
       </collision>
+      <inertial>
+        <mass value="1"/>
+        <origin xyz="0 0 0" rpy="0 0 0"/>
+        <inertia ixx="1" ixy="0" ixz="0" iyy="1" iyz="0" izz="1"/>
+      </inertial>
     </link>
     <link name="${prefix}link_3">
@@ -63,4 +86,9 @@
         </geometry>
       </collision>
+      <inertial>
+        <mass value="1"/>
+        <origin xyz="0 0 0" rpy="0 0 0"/>
+        <inertia ixx="1" ixy="0" ixz="0" iyy="1" iyz="0" izz="1"/>
+      </inertial>
     </link>
     <link name="${prefix}link_4">
@@ -78,4 +106,9 @@
         </geometry>
       </collision>
+      <inertial>
+        <mass value="1"/>
+        <origin xyz="0 0 0" rpy="0 0 0"/>
+        <inertia ixx="1" ixy="0" ixz="0" iyy="1" iyz="0" izz="1"/>
+      </inertial>
     </link>
     <link name="${prefix}link_5">
@@ -93,4 +126,9 @@
         </geometry>
       </collision>
+      <inertial>
+        <mass value="1"/>
+        <origin xyz="0 0 0" rpy="0 0 0"/>
+        <inertia ixx="1" ixy="0" ixz="0" iyy="1" iyz="0" izz="1"/>
+      </inertial>
     </link>
     <link name="${prefix}link_6">
@@ -108,4 +146,9 @@
         </geometry>
       </collision>
+      <inertial>
+        <mass value="1"/>
+        <origin xyz="0 0 0" rpy="0 0 0"/>
+        <inertia ixx="1" ixy="0" ixz="0" iyy="1" iyz="0" izz="1"/>
+      </inertial>
     </link>
     <!-- joints: main serial chain -->

File: denso_ros2_ws/src/Staubli_ROS2-humble/staubli_tx2_60l_moveit_config/config/staubli_tx2_60l.ros2_control.xacro (robot description, xacro)
@@ -1,9 +1,14 @@
 <?xml version="1.0"?>
 <robot xmlns:xacro="http://www.ros.org/wiki/xacro">
-    <xacro:macro name="staubli_tx2_60l_ros2_control" params="name initial_positions_file">
+    <xacro:macro name="staubli_tx2_60l_ros2_control" params="name initial_positions_file sim:=false">
         <xacro:property name="initial_positions" value="${load_yaml(initial_positions_file)['initial_positions']}"/>
         <ros2_control name="${name}" type="system">
             <hardware>
-                <plugin>fake_components/GenericSystem</plugin>
+                <xacro:if value="${sim}">
+                    <plugin>gazebo_ros2_control/GazeboSystem</plugin>
+                </xacro:if>
+                <xacro:unless value="${sim}">
+                    <plugin>fake_components/GenericSystem</plugin>
+                </xacro:unless>
             </hardware>
             <joint name="joint_1">

File: denso_ros2_ws/src/Staubli_ROS2-humble/staubli_tx2_60l_moveit_config/config/staubli_tx2_60l.urdf.xacro (robot description, xacro)
@@ -1,9 +1,17 @@
 <?xml version="1.0"?>
-<robot xmlns:xacro="http://www.ros.org/wiki/xacro" name="staubli">
+<robot xmlns:xacro="http://www.ros.org/wiki/xacro" name="staubli_tx2_60l">
     <xacro:arg name="initial_positions_file" default="initial_positions.yaml" />
-    <!-- Import panda urdf file -->
+    <xacro:arg name="sim" default="true" />
     <xacro:include filename="$(find staubli_tx2_60l_description)/urdf/tx2_60l.xacro" />
-    <!-- Import staubli ros2_control description -->
     <xacro:include filename="staubli_tx2_60l.ros2_control.xacro" />
-    <xacro:staubli_tx2_60l_ros2_control name="StaubliTX260lFakeSystem" initial_positions_file="$(arg initial_positions_file)"/>
+    <xacro:staubli_tx2_60l_ros2_control name="StaubliTX260lSystem" initial_positions_file="$(arg initial_positions_file)" sim="$(arg sim)"/>
+    <xacro:if value="$(arg sim)">
+        <gazebo>
+            <plugin filename="libgazebo_ros2_control.so" name="gazebo_ros2_control">
+                <parameters>$(find staubli_tx2_60l_moveit_config)/config/ros2_controllers.yaml</parameters>
+                <robotParam>robot_description</robotParam>
+                <robotParamNode>robot_state_publisher</robotParamNode>
+            </plugin>
+        </gazebo>
+    </xacro:if>
 </robot>
