Commit message: tx40 running in simulation

File: denso_ros2_ws/src/Staubli_ROS2-humble/staubli_tx2_60l_description/urdf/tx2_60l.xacro (robot description, xacro)
@@ -1,5 +1,10 @@
 <?xml version="1.0" ?>
 <robot name="staubli_tx2_60l" xmlns:xacro="http://wiki.ros.org/xacro">
+  <xacro:arg name="tool" default="none"/>
   <xacro:include filename="$(find staubli_tx2_60l_description)/urdf/tx2_60l_macro.xacro"/>
   <xacro:staubli_tx2_60l prefix=""/>
+  <xacro:unless value="${'$(arg tool)' == 'none'}">
+    <xacro:include filename="$(find tool)/$(arg tool)/$(arg tool).xacro"/>
+    <xacro:call macro="$(arg tool)" namespace="" parent_link="tool0" />
+  </xacro:unless>
 </robot>

File: denso_ros2_ws/src/Staubli_ROS2-humble/staubli_tx2_60l_moveit_config/config/staubli_tx2_60l.ros2_control.xacro (robot description, xacro)
@@ -2,5 +2,5 @@
 <robot xmlns:xacro="http://www.ros.org/wiki/xacro">
     <xacro:macro name="staubli_tx2_60l_ros2_control" params="name initial_positions_file">
-        <xacro:property name="initial_positions" value="${load_yaml(initial_positions_file)['initial_positions']}"/>
+        <xacro:property name="initial_positions" value="${xacro.load_yaml(initial_positions_file)['initial_positions']}"/>
         <ros2_control name="${name}" type="system">
             <hardware>

File: denso_ros2_ws/src/Staubli_ROS2-humble/staubli_tx2_60l_moveit_config/config/staubli_tx2_60l.urdf.xacro (robot description, xacro)
@@ -2,4 +2,5 @@
 <robot xmlns:xacro="http://www.ros.org/wiki/xacro" name="staubli_tx2_60l">
     <xacro:arg name="initial_positions_file" default="initial_positions.yaml" />
+    <xacro:arg name="tool" default="none" />
     <!-- Import panda urdf file -->
     <xacro:include filename="$(find staubli_tx2_60l_description)/urdf/tx2_60l.xacro" />

File: denso_ros2_ws/src/Staubli_ROS2-humble/staubli_tx40_description/urdf/tx40_macro.xacro (robot description, xacro)
@@ -130,5 +130,5 @@
     </joint>
     <joint name="${prefix}joint_3" type="revolute">
-      <origin xyz="0 0 0.255" rpy="0 0 0"/>
+      <origin xyz="0 0 0.225" rpy="0 0 0"/>
       <parent link="${prefix}link_2"/>
       <child link="${prefix}link_3"/>

File: denso_ros2_ws/src/Staubli_ROS2-humble/staubli_tx40_moveit_config/config/staubli_tx40.ros2_control.xacro (robot description, xacro)
@@ -2,5 +2,5 @@
 <robot xmlns:xacro="http://www.ros.org/wiki/xacro">
     <xacro:macro name="staubli_tx40_ros2_control" params="name initial_positions_file">
-        <xacro:property name="initial_positions" value="${load_yaml(initial_positions_file)['initial_positions']}"/>
+        <xacro:property name="initial_positions" value="${xacro.load_yaml(initial_positions_file)['initial_positions']}"/>
         <ros2_control name="${name}" type="system">
             <hardware>

File: denso_ros2_ws/src/Staubli_ROS2-humble/staubli_tx40_moveit_config/config/staubli_tx40.urdf.xacro (robot description, xacro)
@@ -2,8 +2,25 @@
 <robot xmlns:xacro="http://www.ros.org/wiki/xacro" name="staubli_tx40">
     <xacro:arg name="initial_positions_file" default="initial_positions.yaml" />
-    <!-- Import panda urdf file -->
+    <xacro:arg name="tool" default="none" />
+    <xacro:arg name="namespace" default="" />
+    <!-- Robot URDF -->
     <xacro:include filename="$(find staubli_tx40_description)/urdf/tx40.xacro" />
-    <!-- Import staubli ros2_control description -->
+    <!-- ros2_control -->
     <xacro:include filename="staubli_tx40.ros2_control.xacro" />
-    <xacro:staubli_tx40_ros2_control name="StaubliTX260lFakeSystem" initial_positions_file="$(arg initial_positions_file)"/>
+    <xacro:staubli_tx40_ros2_control
+        name="StaubliTX40FakeSystem"
+        initial_positions_file="$(arg initial_positions_file)"/>
+    <!-- Tool dispatcher -->
+    <xacro:if value="${'$(arg tool)' == 'effecteur_v2'}">
+        <xacro:include filename="$(find tool)/effecteur_v2/effecteur_v2.xacro" />
+        <xacro:effecteur_v2 namespace="$(arg namespace)" parent_link="$(arg namespace)tool0" />
+    </xacro:if>
+    <xacro:if value="${'$(arg tool)' == 'effecteur_v1'}">
+        <xacro:include filename="$(find tool)/effecteur_v1/effecteur_v1.xacro" />
+        <xacro:effecteur_v1 namespace="$(arg namespace)" parent_link="$(arg namespace)tool0" />
+    </xacro:if>
+    <xacro:if value="${'$(arg tool)' == 'effecteur_test'}">
+        <xacro:include filename="$(find tool)/effecteur_test/effecteur_test.xacro" />
+        <xacro:effecteur_test namespace="$(arg namespace)" parent_link="$(arg namespace)tool0" />
+    </xacro:if>
 </robot>

File: denso_ros2_ws/src/denso_robot_drivers_ros2/denso_robot_descriptions/urdf/denso_robot.urdf.xacro (robot description, xacro)
@@ -20,9 +20,4 @@
      send_format="$(arg send_format)"
      recv_format="$(arg recv_format)" />
-   <!-- <xacro:unless value="${'$(arg tool)' == 'none'}">
-     <xacro:include filename="$(find denso_robot_descriptions)/tools/$(arg tool)/$(arg tool).xacro"/>
-     <xacro:call macro="$(arg tool)" namespace="$(arg namespace)" parent_link="$(arg namespace)J6" />
-   </xacro:unless>
-    -->
    <xacro:property name="tool_parent_link" value="$(arg namespace)J6" />
    <xacro:if value="${'$(arg model)' == 'hsr065a1_n32'}">
@@ -33,5 +28,5 @@
    </xacro:if>
    <xacro:unless value="${'$(arg tool)' == 'none'}">
-     <xacro:include filename="$(find denso_robot_descriptions)/tools/$(arg tool)/$(arg tool).xacro"/>
+     <xacro:include filename="$(find tool)/$(arg tool)/$(arg tool).xacro"/>
      <xacro:call macro="$(arg tool)" namespace="$(arg namespace)" parent_link="${tool_parent_link}" />
    </xacro:unless>

File: denso_ros2_ws/src/tool/effecteur_test/effecteur_test.xacro (robot description, xacro)
@@ -1,10 +1,10 @@
 <?xml version="1.0"?>
 <robot xmlns:xacro="http://wiki.ros.org/xacro">
-  <xacro:macro name="effecteur_v2" params="namespace parent_link">
+  <xacro:macro name="effecteur_test" params="namespace parent_link">
     <link name="${namespace}tool_link">
       <visual>
-        <origin xyz="0 0 -0.2" rpy="0 0 0" />
+        <origin xyz="0 0 -0.207" rpy="0 0 0" />
         <geometry>
-          <mesh filename="file://$(find denso_robot_descriptions)/tools/effecteur_v2/effecteurV2_visual.stl" scale="0.001 0.001 0.001"/>
+          <mesh filename="file://$(find tool)/effecteur_test/EffecteurTest.STL" scale="0.001 0.001 0.001"/>
         </geometry>
         <material name="grey">
@@ -13,7 +13,7 @@
       </visual>
       <collision>
-        <origin xyz="0 0 -0.2" rpy="0 0 0" />
+        <origin xyz="0 0 -0.207" rpy="0 0 0" />
         <geometry>
-          <mesh filename="file://$(find denso_robot_descriptions)/tools/effecteur_v2/effecteurV2_colision.stl" scale="0.001 0.001 0.001"/>
+          <mesh filename="file://$(find tool)/effecteur_test/EffecteurTest.STL" scale="0.001 0.001 0.001"/>
         </geometry>
       </collision>
@@ -27,5 +27,5 @@
       <parent link="${parent_link}" />
       <child link="${namespace}tool_link" />
-      <origin xyz="0 0 0.2" rpy="0 0 0" />
+      <origin xyz="0 0 0.207" rpy="0 0 0" />
     </joint>
   </xacro:macro>

File: denso_ros2_ws/src/tool/effecteur_v1/effecteur_v1.xacro (robot description, xacro)
@@ -6,5 +6,5 @@
         <origin xyz="0 0 -0.207" rpy="0 0 0" />
         <geometry>
-          <mesh filename="file://$(find denso_robot_descriptions)/tools/effecteur_v1/EffecteurV1.STL" scale="0.001 0.001 0.001"/>
+          <mesh filename="file://$(find tool)/effecteur_v1/EffecteurV1.STL" scale="0.001 0.001 0.001"/>
         </geometry>
         <material name="grey">
@@ -15,5 +15,5 @@
         <origin xyz="0 0 -0.207" rpy="0 0 0" />
         <geometry>
-          <mesh filename="file://$(find denso_robot_descriptions)/tools/effecteur_v1/EffecteurV1.STL" scale="0.001 0.001 0.001"/>
+          <mesh filename="file://$(find tool)/effecteur_v1/EffecteurV1.STL" scale="0.001 0.001 0.001"/>
         </geometry>
       </collision>

File: denso_ros2_ws/src/tool/effecteur_v2/effecteur_v2.xacro (robot description, xacro)
@@ -1,10 +1,10 @@
 <?xml version="1.0"?>
 <robot xmlns:xacro="http://wiki.ros.org/xacro">
-  <xacro:macro name="effecteur_test" params="namespace parent_link">
+  <xacro:macro name="effecteur_v2" params="namespace parent_link">
     <link name="${namespace}tool_link">
       <visual>
-        <origin xyz="0 0 -0.207" rpy="0 0 0" />
+        <origin xyz="0 0 -0.2" rpy="0 0 0" />
         <geometry>
-          <mesh filename="file://$(find denso_robot_descriptions)/tools/effecteur_test/EffecteurTest.STL" scale="0.001 0.001 0.001"/>
+          <mesh filename="file://$(find tool)/effecteur_v2/effecteurV2_visual.stl" scale="0.001 0.001 0.001"/>
         </geometry>
         <material name="grey">
@@ -13,7 +13,7 @@
       </visual>
       <collision>
-        <origin xyz="0 0 -0.207" rpy="0 0 0" />
+        <origin xyz="0 0 -0.2" rpy="0 0 0" />
         <geometry>
-          <mesh filename="file://$(find denso_robot_descriptions)/tools/effecteur_test/EffecteurTest.STL" scale="0.001 0.001 0.001"/>
+          <mesh filename="file://$(find tool)/effecteur_v2/effecteurV2_colision.stl" scale="0.001 0.001 0.001"/>
         </geometry>
       </collision>
@@ -27,5 +27,5 @@
       <parent link="${parent_link}" />
       <child link="${namespace}tool_link" />
-      <origin xyz="0 0 0.207" rpy="0 0 0" />
+      <origin xyz="0 0 0.2" rpy="0 0 0" />
     </joint>
   </xacro:macro>
