Commit message: setting speed and joint limits for vs060 and param for pick_ik

File: denso_ros2_ws/src/denso_robot_drivers_ros2/denso_robot_descriptions/robots/vs060/urdf/denso_robot_joint_limits.xacro (robot description, xacro)
@@ -9,5 +9,5 @@
 			<command_interface name="velocity">
 				<param name="min">0</param>
-				<param name="max">0.392699081698724</param>
+				<param name="max">3</param>
 			</command_interface>
 			<state_interface name="position">
@@ -24,5 +24,5 @@
 			<command_interface name="velocity">
 				<param name="min">0</param>
-				<param name="max">0.261799387799149</param>
+				<param name="max">2</param>
 			</command_interface>
 			<state_interface name="position">
@@ -39,5 +39,5 @@
 			<command_interface name="velocity">
 				<param name="min">0</param>
-				<param name="max">0.285832571599111</param>
+				<param name="max">2</param>
 			</command_interface>
 			<state_interface name="position">
@@ -54,5 +54,5 @@
 			<command_interface name="velocity">
 				<param name="min">0</param>
-				<param name="max">0.392699081698724</param>
+				<param name="max">3</param>
 			</command_interface>
 			<state_interface name="position">
@@ -69,5 +69,5 @@
 			<command_interface name="velocity">
 				<param name="min">0</param>
-				<param name="max">0.302168853397778</param>
+				<param name="max">2</param>
 			</command_interface>
 			<state_interface name="position">
@@ -84,5 +84,5 @@
 			<command_interface name="velocity">
 				<param name="min">0</param>
-				<param name="max">0.628318530717959</param>
+				<param name="max">5</param>
 			</command_interface>
 			<state_interface name="position">

File: denso_ros2_ws/src/denso_robot_drivers_ros2/denso_robot_descriptions/robots/vs060/urdf/denso_robot_kinematics.xacro (robot description, xacro)
@@ -131,5 +131,5 @@
 			<origin rpy="0.000000 0.000000 0.000000" xyz="-0.010000 0.000000 0.164500"/>
 			<axis xyz="-0.000000 -0.000000 1.000000"/>
-			<limit effort="1" lower="-4.71238898038469" upper="4.71238898038469" velocity="3.73064127613788"/>
+			<limit effort="1" lower="-3.14159" upper="3.14159" velocity="3.73064127613788"/>
 			<dynamics damping="0" friction="0"/>
 		</joint>
@@ -185,5 +185,5 @@
 			<origin rpy="0.000000 0.000000 0.000000" xyz="0.000000 0.000000 0.070000"/>
 			<axis xyz="-0.000000 -0.000000 1.000000"/>
-			<limit effort="1" lower="-6.28318530717959" upper="6.28318530717959" velocity="5.96902604182061"/>
+			<limit effort="1" lower="-4.71239" upper="4.71239" velocity="5.96902604182061"/>
 			<dynamics damping="0" friction="0"/>
 		</joint>

Commit message: better planning settings and faster vs060

File: denso_ros2_ws/src/denso_robot_drivers_ros2/denso_robot_descriptions/robots/vs060/urdf/denso_robot_joint_limits.xacro (robot description, xacro)
@@ -9,5 +9,5 @@
 			<command_interface name="velocity">
 				<param name="min">0</param>
-				<param name="max">3</param>
+				<param name="max">8</param>
 			</command_interface>
 			<state_interface name="position">
@@ -24,5 +24,5 @@
 			<command_interface name="velocity">
 				<param name="min">0</param>
-				<param name="max">2</param>
+				<param name="max">5</param>
 			</command_interface>
 			<state_interface name="position">
@@ -39,5 +39,5 @@
 			<command_interface name="velocity">
 				<param name="min">0</param>
-				<param name="max">2</param>
+				<param name="max">6</param>
 			</command_interface>
 			<state_interface name="position">
@@ -54,5 +54,5 @@
 			<command_interface name="velocity">
 				<param name="min">0</param>
-				<param name="max">3</param>
+				<param name="max">9</param>
 			</command_interface>
 			<state_interface name="position">
@@ -69,5 +69,5 @@
 			<command_interface name="velocity">
 				<param name="min">0</param>
-				<param name="max">2</param>
+				<param name="max">7</param>
 			</command_interface>
 			<state_interface name="position">
@@ -84,5 +84,5 @@
 			<command_interface name="velocity">
 				<param name="min">0</param>
-				<param name="max">5</param>
+				<param name="max">15</param>
 			</command_interface>
 			<state_interface name="position">

File: denso_ros2_ws/src/denso_robot_drivers_ros2/denso_robot_descriptions/robots/vs060/urdf/denso_robot_kinematics.xacro (robot description, xacro)
@@ -50,5 +50,5 @@
 			<origin rpy="0.000000 0.000000 0.000000" xyz="0.000000 0.000000 0.181500"/>
 			<axis xyz="-0.000000 -0.000000 1.000000"/>
-			<limit effort="1" lower="-2.96705972839036" upper="2.96705972839036" velocity="3.73064127613788"/>
+			<limit effort="1" lower="-2.96705972839036" upper="2.96705972839036" velocity="8.0"/>
 			<dynamics damping="0" friction="0"/>
 		</joint>
@@ -77,5 +77,5 @@
 			<origin rpy="0.000000 0.000000 0.000000" xyz="0.000000 0.000000 0.163500"/>
 			<axis xyz="-0.000000 1.000000 -0.000000"/>
-			<limit effort="1" lower="-2.0943951023932" upper="2.0943951023932" velocity="2.48709418409192"/>
+			<limit effort="1" lower="-2.0943951023932" upper="2.0943951023932" velocity="5.0"/>
 			<dynamics damping="0" friction="0"/>
 		</joint>
@@ -104,5 +104,5 @@
 			<origin rpy="0.000000 0.000000 0.000000" xyz="0.000000 0.000000 0.305000"/>
 			<axis xyz="-0.000000 1.000000 -0.000000"/>
-			<limit effort="1" lower="-2.18166156499291" upper="2.70526034059121" velocity="2.71540943019156"/>
+			<limit effort="1" lower="-2.18166156499291" upper="2.70526034059121" velocity="6.0"/>
 			<dynamics damping="0" friction="0"/>
 		</joint>
@@ -131,5 +131,5 @@
 			<origin rpy="0.000000 0.000000 0.000000" xyz="-0.010000 0.000000 0.164500"/>
 			<axis xyz="-0.000000 -0.000000 1.000000"/>
-			<limit effort="1" lower="-3.14159" upper="3.14159" velocity="3.73064127613788"/>
+			<limit effort="1" lower="-3.14159" upper="3.14159" velocity="9.0"/>
 			<dynamics damping="0" friction="0"/>
 		</joint>
@@ -158,5 +158,5 @@
 			<origin rpy="0.000000 0.000000 0.000000" xyz="0.000000 0.000000 0.135500"/>
 			<axis xyz="-0.000000 1.000000 -0.000000"/>
-			<limit effort="1" lower="-2.0943951023932" upper="2.0943951023932" velocity="2.87060410727889"/>
+			<limit effort="1" lower="-2.0943951023932" upper="2.0943951023932" velocity="7.0"/>
 			<dynamics damping="0" friction="0"/>
 		</joint>
@@ -185,5 +185,5 @@
 			<origin rpy="0.000000 0.000000 0.000000" xyz="0.000000 0.000000 0.070000"/>
 			<axis xyz="-0.000000 -0.000000 1.000000"/>
-			<limit effort="1" lower="-4.71239" upper="4.71239" velocity="5.96902604182061"/>
+			<limit effort="1" lower="-4.71239" upper="4.71239" velocity="15.0"/>
 			<dynamics damping="0" friction="0"/>
 		</joint>

Commit message: set joint speed and accel for test

File: denso_ros2_ws/src/denso_robot_drivers_ros2/denso_robot_descriptions/robots/vs060/urdf/denso_robot_joint_limits.xacro (robot description, xacro)
@@ -9,5 +9,5 @@
 			<command_interface name="velocity">
 				<param name="min">0</param>
-				<param name="max">8</param>
+				<param name="max">0.392699081698724</param>
 			</command_interface>
 			<state_interface name="position">
@@ -24,5 +24,5 @@
 			<command_interface name="velocity">
 				<param name="min">0</param>
-				<param name="max">5</param>
+				<param name="max">0.261799387799149</param>
 			</command_interface>
 			<state_interface name="position">
@@ -39,5 +39,5 @@
 			<command_interface name="velocity">
 				<param name="min">0</param>
-				<param name="max">6</param>
+				<param name="max">0.285832571599111</param>
 			</command_interface>
 			<state_interface name="position">
@@ -54,5 +54,5 @@
 			<command_interface name="velocity">
 				<param name="min">0</param>
-				<param name="max">9</param>
+				<param name="max">0.392699081698724</param>
 			</command_interface>
 			<state_interface name="position">
@@ -69,5 +69,5 @@
 			<command_interface name="velocity">
 				<param name="min">0</param>
-				<param name="max">7</param>
+				<param name="max">0.302168853397778</param>
 			</command_interface>
 			<state_interface name="position">
@@ -84,5 +84,5 @@
 			<command_interface name="velocity">
 				<param name="min">0</param>
-				<param name="max">15</param>
+				<param name="max">0.628318530717959</param>
 			</command_interface>
 			<state_interface name="position">

File: denso_ros2_ws/src/denso_robot_drivers_ros2/denso_robot_descriptions/robots/vs060/urdf/denso_robot_kinematics.xacro (robot description, xacro)
@@ -50,5 +50,5 @@
 			<origin rpy="0.000000 0.000000 0.000000" xyz="0.000000 0.000000 0.181500"/>
 			<axis xyz="-0.000000 -0.000000 1.000000"/>
-			<limit effort="1" lower="-2.96705972839036" upper="2.96705972839036" velocity="8.0"/>
+			<limit effort="1" lower="-2.96705972839036" upper="2.96705972839036" velocity="3.73064127613788"/>
 			<dynamics damping="0" friction="0"/>
 		</joint>
@@ -77,5 +77,5 @@
 			<origin rpy="0.000000 0.000000 0.000000" xyz="0.000000 0.000000 0.163500"/>
 			<axis xyz="-0.000000 1.000000 -0.000000"/>
-			<limit effort="1" lower="-2.0943951023932" upper="2.0943951023932" velocity="5.0"/>
+			<limit effort="1" lower="-2.0943951023932" upper="2.0943951023932" velocity="2.48709418409192"/>
 			<dynamics damping="0" friction="0"/>
 		</joint>
@@ -104,5 +104,5 @@
 			<origin rpy="0.000000 0.000000 0.000000" xyz="0.000000 0.000000 0.305000"/>
 			<axis xyz="-0.000000 1.000000 -0.000000"/>
-			<limit effort="1" lower="-2.18166156499291" upper="2.70526034059121" velocity="6.0"/>
+			<limit effort="1" lower="-2.18166156499291" upper="2.70526034059121" velocity="2.71540943019156"/>
 			<dynamics damping="0" friction="0"/>
 		</joint>
@@ -131,5 +131,5 @@
 			<origin rpy="0.000000 0.000000 0.000000" xyz="-0.010000 0.000000 0.164500"/>
 			<axis xyz="-0.000000 -0.000000 1.000000"/>
-			<limit effort="1" lower="-3.14159" upper="3.14159" velocity="9.0"/>
+			<limit effort="1" lower="-3.14159" upper="3.14159" velocity="3.73064127613788"/>
 			<dynamics damping="0" friction="0"/>
 		</joint>
@@ -158,5 +158,5 @@
 			<origin rpy="0.000000 0.000000 0.000000" xyz="0.000000 0.000000 0.135500"/>
 			<axis xyz="-0.000000 1.000000 -0.000000"/>
-			<limit effort="1" lower="-2.0943951023932" upper="2.0943951023932" velocity="7.0"/>
+			<limit effort="1" lower="-2.0943951023932" upper="2.0943951023932" velocity="2.87060410727889"/>
 			<dynamics damping="0" friction="0"/>
 		</joint>
@@ -185,5 +185,5 @@
 			<origin rpy="0.000000 0.000000 0.000000" xyz="0.000000 0.000000 0.070000"/>
 			<axis xyz="-0.000000 -0.000000 1.000000"/>
-			<limit effort="1" lower="-4.71239" upper="4.71239" velocity="15.0"/>
+			<limit effort="1" lower="-4.71239" upper="4.71239" velocity="5.96902604182061"/>
 			<dynamics damping="0" friction="0"/>
 		</joint>

Commit message: real robot vs060 speed and accel limits

File: denso_ros2_ws/src/denso_robot_drivers_ros2/denso_robot_descriptions/robots/vs060/urdf/denso_robot_joint_limits.xacro (robot description, xacro)
@@ -9,5 +9,5 @@
 			<command_interface name="velocity">
 				<param name="min">0</param>
-				<param name="max">0.392699081698724</param>
+				<param name="max">3.73064127</param>
 			</command_interface>
 			<state_interface name="position">
@@ -24,5 +24,5 @@
 			<command_interface name="velocity">
 				<param name="min">0</param>
-				<param name="max">0.261799387799149</param>
+				<param name="max">2.48709418</param>
 			</command_interface>
 			<state_interface name="position">
@@ -39,5 +39,5 @@
 			<command_interface name="velocity">
 				<param name="min">0</param>
-				<param name="max">0.285832571599111</param>
+				<param name="max">2.7154094</param>
 			</command_interface>
 			<state_interface name="position">
@@ -54,5 +54,5 @@
 			<command_interface name="velocity">
 				<param name="min">0</param>
-				<param name="max">0.392699081698724</param>
+				<param name="max">3.73064127</param>
 			</command_interface>
 			<state_interface name="position">
@@ -69,5 +69,5 @@
 			<command_interface name="velocity">
 				<param name="min">0</param>
-				<param name="max">0.302168853397778</param>
+				<param name="max">2.87060410</param>
 			</command_interface>
 			<state_interface name="position">
@@ -84,5 +84,5 @@
 			<command_interface name="velocity">
 				<param name="min">0</param>
-				<param name="max">0.628318530717959</param>
+				<param name="max">5.96902604</param>
 			</command_interface>
 			<state_interface name="position">

File: denso_ros2_ws/src/denso_robot_drivers_ros2/denso_robot_descriptions/robots/vs060/urdf/denso_robot_kinematics.xacro (robot description, xacro)
@@ -50,5 +50,5 @@
 			<origin rpy="0.000000 0.000000 0.000000" xyz="0.000000 0.000000 0.181500"/>
 			<axis xyz="-0.000000 -0.000000 1.000000"/>
-			<limit effort="1" lower="-2.96705972839036" upper="2.96705972839036" velocity="3.73064127613788"/>
+			<limit effort="1" lower="-2.96705972839036" upper="2.96705972839036" velocity="3.73064127"/>
 			<dynamics damping="0" friction="0"/>
 		</joint>
@@ -77,5 +77,5 @@
 			<origin rpy="0.000000 0.000000 0.000000" xyz="0.000000 0.000000 0.163500"/>
 			<axis xyz="-0.000000 1.000000 -0.000000"/>
-			<limit effort="1" lower="-2.0943951023932" upper="2.0943951023932" velocity="2.48709418409192"/>
+			<limit effort="1" lower="-2.0943951023932" upper="2.0943951023932" velocity="2.48709418"/>
 			<dynamics damping="0" friction="0"/>
 		</joint>
@@ -104,5 +104,5 @@
 			<origin rpy="0.000000 0.000000 0.000000" xyz="0.000000 0.000000 0.305000"/>
 			<axis xyz="-0.000000 1.000000 -0.000000"/>
-			<limit effort="1" lower="-2.18166156499291" upper="2.70526034059121" velocity="2.71540943019156"/>
+			<limit effort="1" lower="-2.18166156499291" upper="2.70526034059121" velocity="2.7154094"/>
 			<dynamics damping="0" friction="0"/>
 		</joint>
@@ -131,5 +131,5 @@
 			<origin rpy="0.000000 0.000000 0.000000" xyz="-0.010000 0.000000 0.164500"/>
 			<axis xyz="-0.000000 -0.000000 1.000000"/>
-			<limit effort="1" lower="-3.14159" upper="3.14159" velocity="3.73064127613788"/>
+			<limit effort="1" lower="-3.14159" upper="3.14159" velocity="3.73064127"/>
 			<dynamics damping="0" friction="0"/>
 		</joint>
@@ -158,5 +158,5 @@
 			<origin rpy="0.000000 0.000000 0.000000" xyz="0.000000 0.000000 0.135500"/>
 			<axis xyz="-0.000000 1.000000 -0.000000"/>
-			<limit effort="1" lower="-2.0943951023932" upper="2.0943951023932" velocity="2.87060410727889"/>
+			<limit effort="1" lower="-2.0943951023932" upper="2.0943951023932" velocity="2.87060410"/>
 			<dynamics damping="0" friction="0"/>
 		</joint>
@@ -185,5 +185,5 @@
 			<origin rpy="0.000000 0.000000 0.000000" xyz="0.000000 0.000000 0.070000"/>
 			<axis xyz="-0.000000 -0.000000 1.000000"/>
-			<limit effort="1" lower="-4.71239" upper="4.71239" velocity="5.96902604182061"/>
+			<limit effort="1" lower="-4.71239" upper="4.71239" velocity="5.96902604"/>
 			<dynamics damping="0" friction="0"/>
 		</joint>
