Commit message: virtual tool not working

File: ros2_ws/src/mycobot_ros2/mycobot_280/mycobot_280_moveit2/config/firefighter.urdf.xacro (robot description, xacro)
@@ -7,3 +7,9 @@
     <xacro:include filename="firefighter.ros2_control.xacro" />
     <xacro:firefighter_ros2_control name="FakeSystem" initial_positions_file="$(arg initial_positions_file)"/>
+    <link name="tool_tip"/>
+    <joint name="flange_to_tool" type="fixed">
+        <parent link="joint6_flange"/>
+        <child link="tool_tip"/>
+        <origin xyz="0 0 0.10" rpy="0 0 0"/>
+    </joint>
 </robot>

Commit message: tool simulated functional

File: ros2_ws/src/mycobot_ros2/mycobot_280/mycobot_280_moveit2/config/firefighter.urdf.xacro (robot description, xacro)
@@ -7,9 +7,25 @@
     <xacro:include filename="firefighter.ros2_control.xacro" />
     <xacro:firefighter_ros2_control name="FakeSystem" initial_positions_file="$(arg initial_positions_file)"/>
-    <link name="tool_tip"/>
+    <link name="tool_tip">
+      <visual>
+        <origin xyz="0 0 -0.025" rpy="0 0 0"/>
+        <geometry>
+          <cylinder radius="0.015" length="0.05"/>
+        </geometry>
+        <material name="tool_color">
+          <color rgba="0.1 0.1 0.1 1.0"/>
+        </material>
+      </visual>
+      <collision>
+        <origin xyz="0 0 -0.025" rpy="0 0 0"/>
+        <geometry>
+          <cylinder radius="0.015" length="0.05"/>
+        </geometry>
+      </collision>
+    </link>
     <joint name="flange_to_tool" type="fixed">
         <parent link="joint6_flange"/>
         <child link="tool_tip"/>
-        <origin xyz="0 0 0.10" rpy="0 0 0"/>
+        <origin xyz="0 0 0.05" rpy="0 0 0"/>
     </joint>
 </robot>
